Commit message: modified launch file and urdf files for ros2

File: depthai_bridge/urdf/depthai_descr.urdf (robot description, URDF)
Before this commit: robot depthai_camera, 8 links, 7 joints
Links:
- removed link $(arg base_frame)
- removed link $(arg camera_name)_camera_center
- removed link $(arg camera_name)_left_camera_frame
- removed link $(arg camera_name)_left_camera_optical_frame
- removed link $(arg camera_name)_rgb_camera_frame
- removed link $(arg camera_name)_rgb_camera_optical_frame
- removed link $(arg camera_name)_right_camera_frame
- removed link $(arg camera_name)_right_camera_optical_frame
Joints:
- removed joint $(arg camera_name)_center_joint
- removed joint $(arg camera_name)_left_camera_joint
- removed joint $(arg camera_name)_left_camera_optical_joint
- removed joint $(arg camera_name)_rgb_camera_joint
- removed joint $(arg camera_name)_rgb_camera_optical_joint
- removed joint $(arg camera_name)_right_camera_joint
- removed joint $(arg camera_name)_right_camera_optical_joint
