Commit message: Updated Types and URDF and it's launcher

File: depthai_bridge/urdf/depthai_descr.urdf.xacro (robot description, xacro)
@@ -13,5 +13,4 @@
     <xacro:property name="M_PI"     value="3.1415926535897931" />
     <xacro:property name="model"    value="$(arg camera_model)" />
-  <xacro:macro name="camera" >
     <xacro:if value="${model == 'BW1098OAK'}">
     <xacro:property name="baseline" value="0.075" />
@@ -75,4 +74,3 @@
         <child link="$(arg camera_name)_right_camera_optical_frame"/>
     </joint>
-  </xacro:macro>
 </robot>

Commit message: Updated URDF

File: depthai_bridge/urdf/depthai_descr.urdf.xacro (robot description, xacro)
@@ -11,5 +11,5 @@
     <xacro:arg name="cam_yaw"       default="0.0" />
     <xacro:include filename="$(find depthai_bridge)/urdf/include/depthai_macro.urdf.xacro"/>
-    <link name="$(arg base_frame)"/>
-    <xacro:depthai_camera camera_name = "$(arg camera_name)" parent = "$(arg base_frame)" camera_model = "$(arg camera_model)" base_frame = "$(arg base_frame)" cam_pos_x = "$(arg cam_pos_x)" cam_pos_y = "$(arg cam_pos_y)" cam_pos_z = "$(arg cam_pos_z)" cam_roll = "$(arg cam_roll)" cam_pitch = "$(arg cam_pitch)" cam_yaw = "$(arg cam_yaw)"/>
+    <link name="map_base_frame"/>
+    <xacro:depthai_camera camera_name = "$(arg camera_name)" parent = "map_base_frame" camera_model = "$(arg camera_model)" base_frame = "$(arg base_frame)" cam_pos_x = "$(arg cam_pos_x)" cam_pos_y = "$(arg cam_pos_y)" cam_pos_z = "$(arg cam_pos_z)" cam_roll = "$(arg cam_roll)" cam_pitch = "$(arg cam_pitch)" cam_yaw = "$(arg cam_yaw)"/>
 </robot>

File: depthai_bridge/urdf/include/depthai_macro.urdf.xacro (robot description, xacro)
@@ -3,12 +3,17 @@
 <xacro:macro name="depthai_camera" params="camera_name camera_model parent base_frame cam_pos_x cam_pos_y cam_pos_z cam_roll cam_pitch cam_yaw">
     <xacro:property name="M_PI"     value="3.1415926535897931" />
-    <xacro:property name="model"    value="${ camera_model}" />
+    <xacro:property name="model"    value="${camera_model}" />
     <xacro:if value="${model == 'BW1098OAK'}">
         <xacro:property name="baseline" value="0.075" />
     </xacro:if>
     <!-- base_link of the sensor-->
-    <link name="$(arg base_frame)"/>
+    <link name="${base_frame}"/>
+    <joint name="${camera_name}_center_joint" type="fixed">
+        <parent link="${parent}"/>
+        <child link="${base_frame}"/>
+        <origin xyz="${cam_pos_x} ${cam_pos_y} ${cam_pos_z}" rpy="${cam_roll} ${cam_pitch} 1.57" />
+    </joint>
 <!-- device Center -->
-    <link name="${ camera_name}_camera_center">
+    <link name="${camera_name}_model_origin">
         <visual>
             <origin xyz="0 0 0" rpy="0 0 0"/>
@@ -21,47 +26,47 @@
         </visual>
     </link>
-    <joint name="${ camera_name}_center_joint" type="fixed">
-        <parent link="${parent}"/>
-        <child link="${ camera_name}_camera_center"/>
-        <origin xyz="${cam_pos_x} ${cam_pos_y} ${cam_pos_z}" rpy="${cam_roll} ${cam_pitch} 1.57" />
+    <joint name="${camera_name}_model_origin_joint" type="fixed">
+        <parent link="${base_frame}"/>
+        <child link="${camera_name}_model_origin"/>
+        <origin xyz="0 0 0" rpy="1.5708 0 1.5708" />
     </joint>
 <!-- RGB Camera -->
     <link name="${ camera_name}_rgb_camera_frame" />
     <joint name="${ camera_name}_rgb_camera_joint" type="fixed">
-        <parent link="${ camera_name}_camera_center"/>
-        <child link="${ camera_name}_rgb_camera_frame"/>
+        <parent link="${base_frame}"/>
+        <child link="${camera_name}_rgb_camera_frame"/>
         <origin xyz="0 0 0" rpy="0 0 0" />
     </joint>
-    <link name="${ camera_name}_rgb_camera_optical_frame"/>
-    <joint name="${ camera_name}_rgb_camera_optical_joint" type="fixed">
+    <link name="${camera_name}_rgb_camera_optical_frame"/>
+    <joint name="${camera_name}_rgb_camera_optical_joint" type="fixed">
         <origin xyz="0 0 0" rpy="-${M_PI/2} 0.0 -${M_PI/2}"/>
-        <parent link="${ camera_name}_rgb_camera_frame"/>
-        <child link="${ camera_name}_rgb_camera_optical_frame"/>
+        <parent link="${camera_name}_rgb_camera_frame"/>
+        <child link="${camera_name}_rgb_camera_optical_frame"/>
     </joint>
 <!-- Left Camera -->
-    <link name="${ camera_name}_left_camera_frame" />
-    <joint name="${ camera_name}_left_camera_joint" type="fixed">
-        <parent link="${ camera_name}_camera_center"/>
-        <child link="${ camera_name}_left_camera_frame"/>
+    <link name="${camera_name}_left_camera_frame" />
+    <joint name="${camera_name}_left_camera_joint" type="fixed">
+        <parent link="${base_frame}"/>
+        <child link="${camera_name}_left_camera_frame"/>
         <origin xyz="0 ${baseline/2} 0" rpy="0 0 0" />
     </joint>
-    <link name="${ camera_name}_left_camera_optical_frame"/>
-    <joint name="${ camera_name}_left_camera_optical_joint" type="fixed">
+    <link name="${camera_name}_left_camera_optical_frame"/>
+    <joint name="${camera_name}_left_camera_optical_joint" type="fixed">
         <origin xyz="0 0 0" rpy="-${M_PI/2} 0.0 -${M_PI/2}"/>
-        <parent link="${ camera_name}_left_camera_frame"/>
-        <child link="${ camera_name}_left_camera_optical_frame"/>
+        <parent link="${camera_name}_left_camera_frame"/>
+        <child link="${camera_name}_left_camera_optical_frame"/>
     </joint>
 <!-- right Camera -->
-    <link name="${ camera_name}_right_camera_frame" />
-    <joint name="${ camera_name}_right_camera_joint" type="fixed">
-        <parent link="${ camera_name}_camera_center"/>
-        <child link="${ camera_name}_right_camera_frame"/>
+    <link name="${camera_name}_right_camera_frame" />
+    <joint name="${camera_name}_right_camera_joint" type="fixed">
+        <parent link="${base_frame}"/>
+        <child link="${camera_name}_right_camera_frame"/>
         <origin xyz="0 -${baseline/2} 0" rpy="0 0 0" />
     </joint>
-    <link name="${ camera_name}_right_camera_optical_frame"/>
-    <joint name="${ camera_name}_right_camera_optical_joint" type="fixed">
+    <link name="${camera_name}_right_camera_optical_frame"/>
+    <joint name="${camera_name}_right_camera_optical_joint" type="fixed">
         <origin xyz="0 0 0" rpy="-${M_PI/2} 0.0 -${M_PI/2}"/>
-        <parent link="${ camera_name}_right_camera_frame"/>
-        <child link="${ camera_name}_right_camera_optical_frame"/>
+        <parent link="${camera_name}_right_camera_frame"/>
+        <child link="${camera_name}_right_camera_optical_frame"/>
     </joint>
 </xacro:macro>

Commit message: Modified URDF

File: depthai_bridge/urdf/depthai_descr.urdf.xacro (robot description, xacro)
@@ -3,5 +3,5 @@
     <xacro:arg name="camera_name"   default="oak" />
     <xacro:arg name="camera_model"  default="BW1098OAK" />
-    <xacro:arg name="base_frame"    default="base_link" />
+    <xacro:arg name="base_frame"    default="oak-d" />
     <xacro:arg name="cam_pos_x"     default="0.0" />
     <xacro:arg name="cam_pos_y"     default="0.0" />
@@ -10,67 +10,6 @@
     <xacro:arg name="cam_pitch"     default="0.0" />
     <xacro:arg name="cam_yaw"       default="0.0" />
-    <!-- Properties -->
-    <xacro:property name="M_PI"     value="3.1415926535897931" />
-    <xacro:property name="model"    value="$(arg camera_model)" />
-    <xacro:if value="${model == 'BW1098OAK'}">
-    <xacro:property name="baseline" value="0.075" />
-    </xacro:if>
-    <!-- base_link of the sensor-->
-    <link name="$(arg base_frame)" />
-<!-- device Center -->
-    <link name="$(arg camera_name)_camera_center">
-        <visual>
-            <origin xyz="0 0 0" rpy="0 0 0"/>
-            <geometry>
-                <mesh filename="package://depthai_bridge/urdf/models/${model}.dae" />
-            </geometry>
-            <material name="mat">
-                <color rgba="0.8 0.8 0.8 0.8"/>
-            </material>
-        </visual>
-    </link>
-    <joint name="$(arg camera_name)_center_joint" type="fixed">
-        <parent link="$(arg base_frame)"/>
-        <child link="$(arg camera_name)_camera_center"/>
-        <origin xyz="$(arg cam_pos_x) $(arg cam_pos_y) $(arg cam_pos_z)" rpy="$(arg cam_roll) $(arg cam_pitch) $(arg cam_yaw)" />
-    </joint>
-<!-- RGB Camera -->
-    <link name="$(arg camera_name)_rgb_camera_frame" />
-    <joint name="$(arg camera_name)_rgb_camera_joint" type="fixed">
-        <parent link="$(arg base_frame)"/>
-        <child link="$(arg camera_name)_rgb_camera_frame"/>
-        <origin xyz="0 0 0" rpy="0 0 0" />
-    </joint>
-    <link name="$(arg camera_name)_rgb_camera_optical_frame"/>
-    <joint name="$(arg camera_name)_rgb_camera_optical_joint" type="fixed">
-        <origin xyz="0 0 0" rpy="-${M_PI/2} 0.0 -${M_PI/2}"/>
-        <parent link="$(arg camera_name)_rgb_camera_frame"/>
-        <child link="$(arg camera_name)_rgb_camera_optical_frame"/>
-    </joint>
-<!-- Left Camera -->
-    <link name="$(arg camera_name)_left_camera_frame" />
-    <joint name="$(arg camera_name)_left_camera_joint" type="fixed">
-        <parent link="$(arg base_frame)"/>
-        <child link="$(arg camera_name)_left_camera_frame"/>
-        <origin xyz="0 ${baseline/2} 0" rpy="0 0 0" />
-    </joint>
-    <link name="$(arg camera_name)_left_camera_optical_frame"/>
-    <joint name="$(arg camera_name)_left_camera_optical_joint" type="fixed">
-        <origin xyz="0 0 0" rpy="-${M_PI/2} 0.0 -${M_PI/2}"/>
-        <parent link="$(arg camera_name)_left_camera_frame"/>
-        <child link="$(arg camera_name)_left_camera_optical_frame"/>
-    </joint>
-<!-- right Camera -->
-    <link name="$(arg camera_name)_right_camera_frame" />
-    <joint name="$(arg camera_name)_right_camera_joint" type="fixed">
-        <parent link="$(arg base_frame)"/>
-        <child link="$(arg camera_name)_right_camera_frame"/>
-        <origin xyz="0 -${baseline/2} 0" rpy="0 0 0" />
-    </joint>
-    <link name="$(arg camera_name)_right_camera_optical_frame"/>
-    <joint name="$(arg camera_name)_right_camera_optical_joint" type="fixed">
-        <origin xyz="0 0 0" rpy="-${M_PI/2} 0.0 -${M_PI/2}"/>
-        <parent link="$(arg camera_name)_right_camera_frame"/>
-        <child link="$(arg camera_name)_right_camera_optical_frame"/>
-    </joint>
+    <xacro:include filename="$(find depthai_bridge)/urdf/include/depthai_macro.urdf.xacro"/>
+    <link name="map_base_frame"/>
+    <xacro:depthai_camera camera_name = "$(arg camera_name)" parent = "map_base_frame" camera_model = "$(arg camera_model)" base_frame = "$(arg base_frame)" cam_pos_x = "$(arg cam_pos_x)" cam_pos_y = "$(arg cam_pos_y)" cam_pos_z = "$(arg cam_pos_z)" cam_roll = "$(arg cam_roll)" cam_pitch = "$(arg cam_pitch)" cam_yaw = "$(arg cam_yaw)"/>
 </robot>

Commit message: Added argument to urdf launch file so that parent frame can be set in the oak urdf.

File: depthai_bridge/urdf/depthai_descr.urdf.xacro (robot description, xacro)
@@ -4,4 +4,5 @@
     <xacro:arg name="camera_model"  default="BW1098OAK" />
     <xacro:arg name="base_frame"    default="base_link" />
+    <xacro:arg name="parent_frame"  default="base_link" />
     <xacro:arg name="cam_pos_x"     default="0.0" />
     <xacro:arg name="cam_pos_y"     default="0.0" />
@@ -11,5 +12,5 @@
     <xacro:arg name="cam_yaw"       default="0.0" />
     <xacro:include filename="$(find depthai_bridge)/urdf/include/depthai_macro.urdf.xacro"/>
-    <link name="map_base_frame"/>
-    <xacro:depthai_camera camera_name = "$(arg camera_name)" parent = "map_base_frame" camera_model = "$(arg camera_model)" base_frame = "$(arg base_frame)" cam_pos_x = "$(arg cam_pos_x)" cam_pos_y = "$(arg cam_pos_y)" cam_pos_z = "$(arg cam_pos_z)" cam_roll = "$(arg cam_roll)" cam_pitch = "$(arg cam_pitch)" cam_yaw = "$(arg cam_yaw)"/>
+    <link name="$(arg parent_frame)"/>
+    <xacro:depthai_camera camera_name = "$(arg camera_name)" parent = "$(arg parent_frame)" camera_model = "$(arg camera_model)" base_frame = "$(arg base_frame)" cam_pos_x = "$(arg cam_pos_x)" cam_pos_y = "$(arg cam_pos_y)" cam_pos_z = "$(arg cam_pos_z)" cam_roll = "$(arg cam_roll)" cam_pitch = "$(arg cam_pitch)" cam_yaw = "$(arg cam_yaw)"/>
 </robot>

Commit message: Updated the urdf launch file of ROS2

File: depthai_bridge/urdf/depthai_descr.urdf.xacro (robot description, xacro)
@@ -2,7 +2,7 @@
 <robot name="depthai_camera" xmlns:xacro="http://ros.org/wiki/xacro">
     <xacro:arg name="camera_name"   default="oak" />
-    <xacro:arg name="camera_model"  default="BW1098OAK" />
-    <xacro:arg name="base_frame"    default="base_link" />
-    <xacro:arg name="parent_frame"  default="base_link" />
+    <xacro:arg name="camera_model"  default="OAK-D" />
+    <xacro:arg name="base_frame"    default="oak-d_frame" />
+    <xacro:arg name="parent_frame"  default="oak-d-base-frame" />
     <xacro:arg name="cam_pos_x"     default="0.0" />
     <xacro:arg name="cam_pos_y"     default="0.0" />

File: depthai_bridge/urdf/include/depthai_macro.urdf.xacro (robot description, xacro)
@@ -6,5 +6,5 @@
     <!-- <xacro:if value="${model == 'BW1098OAK'}">
     </xacro:if> -->
-    <xacro:property name="baseline" value="0.095" />
+    <xacro:property name="baseline" value="0.075" />
     <!-- base_link of the sensor-->
     <link name="${base_frame}"/>

Commit message: change camera_name parameter to tf_prefix

File: depthai_bridge/urdf/depthai_descr.urdf.xacro (robot description, xacro)
@@ -1,5 +1,5 @@
 <?xml version="1.0"?>
 <robot name="depthai_camera" xmlns:xacro="http://ros.org/wiki/xacro">
-    <xacro:arg name="camera_name"   default="oak" />
+    <xacro:arg name="tf_prefix"     default="oak" />
     <xacro:arg name="camera_model"  default="OAK-D" />
     <xacro:arg name="base_frame"    default="oak-d_frame" />
@@ -13,4 +13,4 @@
     <xacro:include filename="$(find depthai_bridge)/urdf/include/depthai_macro.urdf.xacro"/>
     <link name="$(arg parent_frame)"/>
-    <xacro:depthai_camera camera_name = "$(arg camera_name)" parent = "$(arg parent_frame)" camera_model = "$(arg camera_model)" base_frame = "$(arg base_frame)" cam_pos_x = "$(arg cam_pos_x)" cam_pos_y = "$(arg cam_pos_y)" cam_pos_z = "$(arg cam_pos_z)" cam_roll = "$(arg cam_roll)" cam_pitch = "$(arg cam_pitch)" cam_yaw = "$(arg cam_yaw)"/>
+    <xacro:depthai_camera tf_prefix= "$(arg tf_prefix)" parent = "$(arg parent_frame)" camera_model = "$(arg camera_model)" base_frame = "$(arg base_frame)" cam_pos_x = "$(arg cam_pos_x)" cam_pos_y = "$(arg cam_pos_y)" cam_pos_z = "$(arg cam_pos_z)" cam_roll = "$(arg cam_roll)" cam_pitch = "$(arg cam_pitch)" cam_yaw = "$(arg cam_yaw)"/>
 </robot>

File: depthai_bridge/urdf/include/depthai_macro.urdf.xacro (robot description, xacro)
@@ -1,5 +1,5 @@
 <?xml version="1.0"?>
 <robot name="depthai_camera" xmlns:xacro="http://ros.org/wiki/xacro">
-<xacro:macro name="depthai_camera" params="camera_name camera_model parent base_frame cam_pos_x cam_pos_y cam_pos_z cam_roll cam_pitch cam_yaw">
+<xacro:macro name="depthai_camera" params="tf_prefix camera_model parent base_frame cam_pos_x cam_pos_y cam_pos_z cam_roll cam_pitch cam_yaw">
     <xacro:property name="M_PI"     value="3.1415926535897931" />
     <xacro:property name="model"    value="${camera_model}" />
@@ -9,5 +9,5 @@
     <!-- base_link of the sensor-->
     <link name="${base_frame}"/>
-    <joint name="${camera_name}_center_joint" type="fixed">
+    <joint name="${tf_prefix}_center_joint" type="fixed">
         <parent link="${parent}"/>
         <child link="${base_frame}"/>
@@ -15,5 +15,5 @@
     </joint>
 <!-- device Center -->
-    <link name="${camera_name}_model_origin">
+    <link name="${tf_prefix}_model_origin">
         <visual>
             <origin xyz="0 0 0" rpy="0 0 0"/>
@@ -26,54 +26,54 @@
         </visual>
     </link>
-    <joint name="${camera_name}_model_origin_joint" type="fixed">
+    <joint name="${tf_prefix}_model_origin_joint" type="fixed">
         <parent link="${base_frame}"/>
-        <child link="${camera_name}_model_origin"/>
+        <child link="${tf_prefix}_model_origin"/>
         <origin xyz="0 0 0" rpy="1.5708 0 1.5708" />
     </joint>
 <!-- IMU -->
-    <link name="${ camera_name}_imu_frame" />
-    <joint name="${ camera_name}_imu_joint" type="fixed">
+    <link name="${ tf_prefix}_imu_frame" />
+    <joint name="${ tf_prefix}_imu_joint" type="fixed">
         <parent link="${base_frame}"/>
-        <child link="${camera_name}_imu_frame"/>
+        <child link="${tf_prefix}_imu_frame"/>
         <origin xyz="0 0 0" rpy="-${M_PI/2} 0 -${M_PI/2}" />
     </joint>
 <!-- RGB Camera -->
-    <link name="${ camera_name}_rgb_camera_frame" />
-    <joint name="${ camera_name}_rgb_camera_joint" type="fixed">
+    <link name="${ tf_prefix}_rgb_camera_frame" />
+    <joint name="${ tf_prefix}_rgb_camera_joint" type="fixed">
         <parent link="${base_frame}"/>
-        <child link="${camera_name}_rgb_camera_frame"/>
+        <child link="${tf_prefix}_rgb_camera_frame"/>
         <origin xyz="0 0 0" rpy="0 0 0" />
     </joint>
-    <link name="${camera_name}_rgb_camera_optical_frame"/>
-    <joint name="${camera_name}_rgb_camera_optical_joint" type="fixed">
+    <link name="${tf_prefix}_rgb_camera_optical_frame"/>
+    <joint name="${tf_prefix}_rgb_camera_optical_joint" type="fixed">
         <origin xyz="0 0 0" rpy="-${M_PI/2} 0.0 -${M_PI/2}"/>
-        <parent link="${camera_name}_rgb_camera_frame"/>
-        <child link="${camera_name}_rgb_camera_optical_frame"/>
+        <parent link="${tf_prefix}_rgb_camera_frame"/>
+        <child link="${tf_prefix}_rgb_camera_optical_frame"/>
     </joint>
 <!-- Left Camera -->
-    <link name="${camera_name}_left_camera_frame" />
-    <joint name="${camera_name}_left_camera_joint" type="fixed">
+    <link name="${tf_prefix}_left_camera_frame" />
+    <joint name="${tf_prefix}_left_camera_joint" type="fixed">
         <parent link="${base_frame}"/>
-        <child link="${camera_name}_left_camera_frame"/>
+        <child link="${tf_prefix}_left_camera_frame"/>
         <origin xyz="0 ${baseline/2} 0" rpy="0 0 0" />
     </joint>
-    <link name="${camera_name}_left_camera_optical_frame"/>
-    <joint name="${camera_name}_left_camera_optical_joint" type="fixed">
+    <link name="${tf_prefix}_left_camera_optical_frame"/>
+    <joint name="${tf_prefix}_left_camera_optical_joint" type="fixed">
         <origin xyz="0 0 0" rpy="-${M_PI/2} 0.0 -${M_PI/2}"/>
-        <parent link="${camera_name}_left_camera_frame"/>
-        <child link="${camera_name}_left_camera_optical_frame"/>
+        <parent link="${tf_prefix}_left_camera_frame"/>
+        <child link="${tf_prefix}_left_camera_optical_frame"/>
     </joint>
 <!-- right Camera -->
-    <link name="${camera_name}_right_camera_frame" />
-    <joint name="${camera_name}_right_camera_joint" type="fixed">
+    <link name="${tf_prefix}_right_camera_frame" />
+    <joint name="${tf_prefix}_right_camera_joint" type="fixed">
         <parent link="${base_frame}"/>
-        <child link="${camera_name}_right_camera_frame"/>
+        <child link="${tf_prefix}_right_camera_frame"/>
         <origin xyz="0 -${baseline/2} 0" rpy="0 0 0" />
     </joint>
-    <link name="${camera_name}_right_camera_optical_frame"/>
-    <joint name="${camera_name}_right_camera_optical_joint" type="fixed">
+    <link name="${tf_prefix}_right_camera_optical_frame"/>
+    <joint name="${tf_prefix}_right_camera_optical_joint" type="fixed">
         <origin xyz="0 0 0" rpy="-${M_PI/2} 0.0 -${M_PI/2}"/>
-        <parent link="${camera_name}_right_camera_frame"/>
-        <child link="${camera_name}_right_camera_optical_frame"/>
+        <parent link="${tf_prefix}_right_camera_frame"/>
+        <child link="${tf_prefix}_right_camera_optical_frame"/>
     </joint>
 </xacro:macro>
