Commit message: WIP rae urdf model

File: depthai_bridge/urdf/rae.urdf.xacro (robot description, xacro)
@@ -1,8 +1,9 @@
 <?xml version="1.0"?>
 <robot name="rae" xmlns:xacro="http://ros.org/wiki/xacro">
+    <link name="base_frame"/>
     <link name="chassis">
       <inertial>
         <mass value="1.0"/>
-        <origin rpy="0 0 0" xyz="0 0 0"/>
+        <origin rpy="0.0 0.0 0.0" xyz="0.0 0.0 0.0"/>
         <inertia
           ixx = "0.166667"
@@ -21,14 +22,27 @@
       </collision>
       <visual>
-        <origin rpy="0.049227 0.011061 0.000747" xyz="-0 -1e-06 3.14159"/>
+        <origin rpy="0.0 0.0 0.0" xyz="0.0 0.0 0.0"/>
         <geometry>
           <mesh filename="package://depthai_bridge/urdf/models/rae_chassis.stl" scale="1.0 1.0 1.0"/>
         </geometry>
+        <material name="mat">
+          <lighting>1</lighting>
+          <!-- <color rgba="0.1 0.1 0.1 1.0"/> -->
+          <shader type='pixel'/>
+          <emissive>0 0 0 1</emissive>
+        </material>
+        <transparency>0</transparency>
+        <cast_shadows>1</cast_shadows>
       </visual>
     </link>
+    <joint name="base_chassis_joint" type="fixed">
+        <parent link="base_frame"/>
+        <child link="chassis"/>
+        <origin rpy="1.57 0.0 1.57" xyz="0.0 0.0 0.0" />
+    </joint>
     <link name="left_wheel">
       <inertial>
         <mass value="1.0"/>
-        <origin rpy="-0 -1e-06 3.14159" xyz="0.049227 0.011061 0.000747"/>
+        <origin rpy="0.0 0.0 0.0" xyz="0.0 0.0 0.0"/>
         <inertia
           ixx = "0.166667"
@@ -56,5 +70,5 @@
       <inertial>
         <mass value="1.0"/>
-        <origin rpy="0 0 0" xyz="-0.048887 0.00846 0.000728"/>
+        <origin rpy="0.0 0.0 0.0" xyz="0.0 0.0 0.0"/>
         <inertia
           ixx = "0.166667"
@@ -80,5 +94,5 @@
     </link>
     <joint name='left_wheel_hinge' type='revolute'>
-      <origin rpy="0.0 0.0 0.0 " xyz="0.0 0.0 0.0"/>
+      <origin rpy="0.0 0.0 0.0 " xyz="-0.0497 0.00518 -0.03048"/>
       <child  link="left_wheel"/>
       <parent link="chassis"/>
@@ -87,5 +101,5 @@
     </joint>
     <joint name='right_wheel_hinge' type='revolute'>
-      <origin rpy="0.0 0.0 0.0 " xyz="0.0 0.0 0.0"/>
+      <origin rpy="0.0 3.14159 0.0 " xyz="0.0497 0.00518 -0.03048"/>
       <child  link="right_wheel"/>
       <parent link="chassis"/>

Commit message: added rae-urdf

File: depthai_bridge/urdf/rae.urdf.xacro (robot description, xacro)
@@ -1,4 +1,5 @@
 <?xml version="1.0"?>
 <robot name="rae" xmlns:xacro="http://ros.org/wiki/xacro">
+    <link name="base_frame"/>
     <link name="chassis">
       <inertial>
@@ -79,4 +80,9 @@
       </visual>
     </link>
+    <joint name="base_joint" type="fixed">
+        <parent link="base_frame"/>
+        <child link="chassis"/>
+        <origin xyz="0 0 0" rpy="0 0 0" />
+    </joint>
     <joint name='left_wheel_hinge' type='revolute'>
       <origin rpy="0.0 0.0 0.0 " xyz="0.0 0.0 0.0"/>
