Commit message: fix yaw

File: depthai_bridge/urdf/include/depthai_macro.urdf.xacro (robot description, xacro)
@@ -12,5 +12,5 @@
         <parent link="${parent}"/>
         <child link="${base_frame}"/>
-        <origin xyz="${cam_pos_x} ${cam_pos_y} ${cam_pos_z}" rpy="${cam_roll} ${cam_pitch} 1.57" />
+        <origin xyz="${cam_pos_x} ${cam_pos_y} ${cam_pos_z}" rpy="${cam_roll} ${cam_pitch} ${cam_yaw}" />
     </joint>
 <!-- device Center -->

Commit message: Added IMU support

File: depthai_bridge/urdf/include/depthai_macro.urdf.xacro (robot description, xacro)
@@ -30,4 +30,11 @@
         <child link="${camera_name}_model_origin"/>
         <origin xyz="0 0 0" rpy="1.5708 0 1.5708" />
+    </joint>
+<!-- IMU -->
+    <link name="${ camera_name}_imu_frame" />
+    <joint name="${ camera_name}_imu_joint" type="fixed">
+        <parent link="${base_frame}"/>
+        <child link="${camera_name}_imu_frame"/>
+        <origin xyz="0 0 0" rpy="-${M_PI/2} 0 -${M_PI/2}" />
     </joint>
 <!-- RGB Camera -->

Commit message: Fixing size of stl files and some modifications in reading them.

File: depthai_bridge/urdf/include/depthai_macro.urdf.xacro (robot description, xacro)
@@ -4,7 +4,7 @@
     <xacro:property name="M_PI"     value="3.1415926535897931" />
     <xacro:property name="model"    value="${camera_model}" />
-    <xacro:if value="${model == 'BW1098OAK'}">
-        <xacro:property name="baseline" value="0.075" />
-    </xacro:if>
+    <!-- <xacro:if value="${model == 'BW1098OAK'}">
+    </xacro:if> -->
+    <xacro:property name="baseline" value="0.095" />
     <!-- base_link of the sensor-->
     <link name="${base_frame}"/>
@@ -19,5 +19,5 @@
             <origin xyz="0 0 0" rpy="0 0 0"/>
             <geometry>
-                <mesh filename="package://depthai_bridge/urdf/models/${model}.dae" />
+                <mesh filename="package://depthai_bridge/urdf/models/${model}.stl" />
             </geometry>
             <material name="mat">

Commit message: Change camera_name parameter to tf_prefix and fix URDF launch for ROS1 (#67)
* change camera_name parameter to tf_prefix

* fix urdf for ros1

* revert URDF changes

Co-authored-by: Sachin Guruswamy <43363595+saching13@users.noreply.github.com>

File: depthai_bridge/urdf/include/depthai_macro.urdf.xacro (robot description, xacro)
@@ -32,6 +32,6 @@
     </joint>
 <!-- IMU -->
-    <link name="${ camera_name}_imu_frame" />
-    <joint name="${ camera_name}_imu_joint" type="fixed">
+    <link name="${camera_name}_imu_frame" />
+    <joint name="${camera_name}_imu_joint" type="fixed">
         <parent link="${base_frame}"/>
         <child link="${camera_name}_imu_frame"/>
@@ -39,6 +39,6 @@
     </joint>
 <!-- RGB Camera -->
-    <link name="${ camera_name}_rgb_camera_frame" />
-    <joint name="${ camera_name}_rgb_camera_joint" type="fixed">
+    <link name="${camera_name}_rgb_camera_frame" />
+    <joint name="${camera_name}_rgb_camera_joint" type="fixed">
         <parent link="${base_frame}"/>
         <child link="${camera_name}_rgb_camera_frame"/>

Commit message: Added IMU pos WIP

File: depthai_bridge/urdf/include/depthai_macro.urdf.xacro (robot description, xacro)
@@ -7,4 +7,12 @@
     </xacro:if> -->
     <xacro:property name="baseline" value="0.075" />
+    <xacro:if value="${model == 'OAK-D'}">
+      <xacro:property name="imu_offset_x" value="0.015" />
+      <xacro:property name="imu_offset_y" value="-0.013662" />
+      <xacro:property name="imu_offset_z" value="0" />
+      <xacro:property name="imu_r" value="0.0" />
+      <xacro:property name="imu_p" value="0.0" />
+      <xacro:property name="imu_y" value="0.0" />
+    </xacro:if>
     <!-- base_link of the sensor-->
     <link name="${base_frame}"/>

Commit message: Verified time stamps, Included position of IMU in OAK-D, added GYRO interpolation

File: depthai_bridge/urdf/include/depthai_macro.urdf.xacro (robot description, xacro)
@@ -8,10 +8,10 @@
     <xacro:property name="baseline" value="0.075" />
     <xacro:if value="${model == 'OAK-D'}">
-      <xacro:property name="imu_offset_x" value="0.015" />
-      <xacro:property name="imu_offset_y" value="-0.013662" />
-      <xacro:property name="imu_offset_z" value="0" />
-      <xacro:property name="imu_r" value="0.0" />
-      <xacro:property name="imu_p" value="0.0" />
-      <xacro:property name="imu_y" value="0.0" />
+      <xacro:property name="imu_offset_x" value="0.0" />
+      <xacro:property name="imu_offset_y" value="-0.015" />
+      <xacro:property name="imu_offset_z" value="-0.013662" />
+      <xacro:property name="imu_r" value="0" />
+      <xacro:property name="imu_p" value="1.5708" />
+      <xacro:property name="imu_y" value="0" />
     </xacro:if>
     <!-- base_link of the sensor-->
@@ -44,5 +44,5 @@
         <parent link="${base_frame}"/>
         <child link="${camera_name}_imu_frame"/>
-        <origin xyz="0 0 0" rpy="-${M_PI/2} 0 -${M_PI/2}" />
+        <origin xyz="${imu_offset_x} ${imu_offset_y} ${imu_offset_z}" rpy="${imu_r} ${imu_p} ${imu_y}" />
     </joint>
 <!-- RGB Camera -->

Commit message: Imu interpolation (#90)
* Added workflow on devel too (#81)

* Fix interpolation

* WIP updated Bridge publisher

* Devel (#83)

* Added workflow on devel too

* Timestamp update (#80)

* Updated depthai to use timestamp from 2.15 of DepthAI

* Upgrade version:

* Add depthai version check for upgrade

* Refactored Bridge Publisher, Image Converter and Disparity converter

* Updated Image Detection and Spatial Image detection converter

* WIP Interpolation function

* Created united IMU message TIME step WIP"
:

* Added utility and Implemented Double conversion in Milli Seconds

* Fixinh bugs WIP1

* Working INterpolation

* Working interpolation of Accel to gyro at 400Hz. Interpolating Gyro to Accel pending

* Added IMU pos WIP

* Verified time stamps, Included position of IMU in OAK-D, added GYRO interpolation

* Updated logging Macros

* Included IMU copy mode

* Bug Fixes

* Fix styling

* Style fixing 2:

File: depthai_bridge/urdf/include/depthai_macro.urdf.xacro (robot description, xacro)
@@ -7,4 +7,12 @@
     </xacro:if> -->
     <xacro:property name="baseline" value="0.075" />
+    <xacro:if value="${model == 'OAK-D'}">
+      <xacro:property name="imu_offset_x" value="0.0" />
+      <xacro:property name="imu_offset_y" value="-0.015" />
+      <xacro:property name="imu_offset_z" value="-0.013662" />
+      <xacro:property name="imu_r" value="0" />
+      <xacro:property name="imu_p" value="1.5708" />
+      <xacro:property name="imu_y" value="0" />
+    </xacro:if>
     <!-- base_link of the sensor-->
     <link name="${base_frame}"/>
@@ -36,5 +44,5 @@
         <parent link="${base_frame}"/>
         <child link="${camera_name}_imu_frame"/>
-        <origin xyz="0 0 0" rpy="-${M_PI/2} 0 -${M_PI/2}" />
+        <origin xyz="${imu_offset_x} ${imu_offset_y} ${imu_offset_z}" rpy="${imu_r} ${imu_p} ${imu_y}" />
     </joint>
 <!-- RGB Camera -->

Commit message: Added rgba params to depthai_camera macro

File: depthai_bridge/urdf/include/depthai_macro.urdf.xacro (robot description, xacro)
@@ -1,5 +1,8 @@
 <?xml version="1.0"?>
 <robot name="depthai_camera" xmlns:xacro="http://ros.org/wiki/xacro">
-<xacro:macro name="depthai_camera" params="camera_name camera_model parent base_frame cam_pos_x cam_pos_y cam_pos_z cam_roll cam_pitch cam_yaw">
+<xacro:macro name="depthai_camera" params="camera_name camera_model parent base_frame
+                                           cam_pos_x cam_pos_y cam_pos_z
+                                           cam_roll cam_pitch cam_yaw
+                                           r:=0.8 g:=0.8 b:=0.8 a:=0.8">
     <xacro:property name="M_PI"     value="3.1415926535897931" />
     <xacro:property name="model"    value="${camera_model}" />
@@ -22,5 +25,5 @@
             </geometry>
             <material name="mat">
-                <color rgba="0.8 0.8 0.8 0.8"/>
+                <color rgba="${r} ${g} ${b} ${a}"/>
             </material>
         </visual>

Commit message: Added rgba params to depthai_camera macro (#91)

File: depthai_bridge/urdf/include/depthai_macro.urdf.xacro (robot description, xacro)
@@ -1,5 +1,8 @@
 <?xml version="1.0"?>
 <robot name="depthai_camera" xmlns:xacro="http://ros.org/wiki/xacro">
-<xacro:macro name="depthai_camera" params="camera_name camera_model parent base_frame cam_pos_x cam_pos_y cam_pos_z cam_roll cam_pitch cam_yaw">
+<xacro:macro name="depthai_camera" params="camera_name camera_model parent base_frame
+                                           cam_pos_x cam_pos_y cam_pos_z
+                                           cam_roll cam_pitch cam_yaw
+                                           r:=0.8 g:=0.8 b:=0.8 a:=0.8">
     <xacro:property name="M_PI"     value="3.1415926535897931" />
     <xacro:property name="model"    value="${camera_model}" />
@@ -30,5 +33,5 @@
             </geometry>
             <material name="mat">
-                <color rgba="0.8 0.8 0.8 0.8"/>
+                <color rgba="${r} ${g} ${b} ${a}"/>
             </material>
         </visual>

Commit message: fix #96: Set up IMU frames only for cameras with IMU

File: depthai_bridge/urdf/include/depthai_macro.urdf.xacro (robot description, xacro)
@@ -7,8 +7,10 @@
     <xacro:property name="M_PI"     value="3.1415926535897931" />
     <xacro:property name="model"    value="${camera_model}" />
+    <xacro:property name="has_imu" value="false" />
     <!-- <xacro:if value="${model == 'BW1098OAK'}">
     </xacro:if> -->
     <xacro:property name="baseline" value="0.075" />
     <xacro:if value="${model == 'OAK-D'}">
+      <xacro:property name="has_imu" value="true" />
       <xacro:property name="imu_offset_x" value="0.0" />
       <xacro:property name="imu_offset_y" value="-0.015" />
@@ -42,11 +44,13 @@
         <origin xyz="0 0 0" rpy="1.5708 0 1.5708" />
     </joint>
+    <xacro:if value="${has_imu}">
 <!-- IMU -->
-    <link name="${camera_name}_imu_frame" />
-    <joint name="${camera_name}_imu_joint" type="fixed">
-        <parent link="${base_frame}"/>
-        <child link="${camera_name}_imu_frame"/>
-        <origin xyz="${imu_offset_x} ${imu_offset_y} ${imu_offset_z}" rpy="${imu_r} ${imu_p} ${imu_y}" />
-    </joint>
+        <link name="${camera_name}_imu_frame" />
+        <joint name="${camera_name}_imu_joint" type="fixed">
+            <parent link="${base_frame}"/>
+            <child link="${camera_name}_imu_frame"/>
+            <origin xyz="${imu_offset_x} ${imu_offset_y} ${imu_offset_z}" rpy="${imu_r} ${imu_p} ${imu_y}" />
+        </joint>
+    </xacro:if>
 <!-- RGB Camera -->
     <link name="${camera_name}_rgb_camera_frame" />
