Commit message: update urdfs

File: depthai_descriptions/urdf/depthai_descr.urdf.xacro (robot description, xacro)
@@ -11,6 +11,7 @@
     <xacro:arg name="cam_pitch"     default="0.0" />
     <xacro:arg name="cam_yaw"       default="0.0" />
+    <xacro:arg name="is_bno"        default="false"/>
     <xacro:include filename="$(find depthai_descriptions)/urdf/include/depthai_macro.urdf.xacro"/>
     <link name="$(arg parent_frame)"/>
-    <xacro:depthai_camera camera_name = "$(arg camera_name)" parent = "$(arg parent_frame)" camera_model = "$(arg camera_model)" base_frame = "$(arg base_frame)" cam_pos_x = "$(arg cam_pos_x)" cam_pos_y = "$(arg cam_pos_y)" cam_pos_z = "$(arg cam_pos_z)" cam_roll = "$(arg cam_roll)" cam_pitch = "$(arg cam_pitch)" cam_yaw = "$(arg cam_yaw)"/>
+    <xacro:depthai_camera camera_name = "$(arg camera_name)" parent = "$(arg parent_frame)" camera_model = "$(arg camera_model)" base_frame = "$(arg base_frame)" cam_pos_x = "$(arg cam_pos_x)" cam_pos_y = "$(arg cam_pos_y)" cam_pos_z = "$(arg cam_pos_z)" cam_roll = "$(arg cam_roll)" cam_pitch = "$(arg cam_pitch)" cam_yaw = "$(arg cam_yaw)" is_bno = "$(arg is_bno)"/>
 </robot>

File: depthai_descriptions/urdf/include/depthai_macro.urdf.xacro (robot description, xacro)
@@ -3,9 +3,10 @@
 <xacro:macro name="depthai_camera" params="camera_name camera_model parent base_frame
                                            cam_pos_x cam_pos_y cam_pos_z
-                                           cam_roll cam_pitch cam_yaw
+                                           cam_roll cam_pitch cam_yaw is_bno
                                            r:=0.8 g:=0.8 b:=0.8 a:=0.8">
     <xacro:property name="M_PI"     value="3.1415926535897931" />
     <xacro:property name="model"    value="${camera_model}" />
     <xacro:property name="has_imu" value="false" />
+    <xacro:property name="is_bno" value="false"/>
     <!-- <xacro:if value="${model == 'BW1098OAK'}">
     </xacro:if> -->
@@ -19,4 +20,24 @@
       <xacro:property name="imu_p" value="1.5708" />
       <xacro:property name="imu_y" value="0" />
+    </xacro:if>
+    <xacro:if value="${model == 'OAK-D-PRO-W'}">
+      <xacro:if value="${is_bno}">
+        <xacro:property name="has_imu" value="true" />
+        <xacro:property name="imu_offset_x" value="0.075448" />
+        <xacro:property name="imu_offset_y" value="0.0079" />
+        <xacro:property name="imu_offset_z" value="0.0" />
+        <xacro:property name="imu_r" value="-3.1415" />
+        <xacro:property name="imu_p" value="0.0" />
+        <xacro:property name="imu_y" value="-1.5708" />
+      </xacro:if>
+      <xacro:unless value="${is_bno}">
+        <xacro:property name="has_imu" value="true" />
+        <xacro:property name="imu_offset_x" value="0.06935" />
+        <xacro:property name="imu_offset_y" value="0.00231" />
+        <xacro:property name="imu_offset_z" value="0.0" />
+        <xacro:property name="imu_r" value="-3.1415" />
+        <xacro:property name="imu_p" value="0.0" />
+        <xacro:property name="imu_y" value="-1.5708" />
+      </xacro:unless>
     </xacro:if>
     <!-- base_link of the sensor-->

Commit message: remove bno quick fix

File: depthai_descriptions/urdf/depthai_descr.urdf.xacro (robot description, xacro)
@@ -11,7 +11,6 @@
     <xacro:arg name="cam_pitch"     default="0.0" />
     <xacro:arg name="cam_yaw"       default="0.0" />
-    <xacro:arg name="is_bno"        default="false"/>
     <xacro:include filename="$(find depthai_descriptions)/urdf/include/depthai_macro.urdf.xacro"/>
     <link name="$(arg parent_frame)"/>
-    <xacro:depthai_camera camera_name = "$(arg camera_name)" parent = "$(arg parent_frame)" camera_model = "$(arg camera_model)" base_frame = "$(arg base_frame)" cam_pos_x = "$(arg cam_pos_x)" cam_pos_y = "$(arg cam_pos_y)" cam_pos_z = "$(arg cam_pos_z)" cam_roll = "$(arg cam_roll)" cam_pitch = "$(arg cam_pitch)" cam_yaw = "$(arg cam_yaw)" is_bno = "$(arg is_bno)"/>
+    <xacro:depthai_camera camera_name = "$(arg camera_name)" parent = "$(arg parent_frame)" camera_model = "$(arg camera_model)" base_frame = "$(arg base_frame)" cam_pos_x = "$(arg cam_pos_x)" cam_pos_y = "$(arg cam_pos_y)" cam_pos_z = "$(arg cam_pos_z)" cam_roll = "$(arg cam_roll)" cam_pitch = "$(arg cam_pitch)" cam_yaw = "$(arg cam_yaw)"/>
 </robot>

File: depthai_descriptions/urdf/include/depthai_macro.urdf.xacro (robot description, xacro)
@@ -3,10 +3,9 @@
 <xacro:macro name="depthai_camera" params="camera_name camera_model parent base_frame
                                            cam_pos_x cam_pos_y cam_pos_z
-                                           cam_roll cam_pitch cam_yaw is_bno
+                                           cam_roll cam_pitch cam_yaw
                                            r:=0.8 g:=0.8 b:=0.8 a:=0.8">
     <xacro:property name="M_PI"     value="3.1415926535897931" />
     <xacro:property name="model"    value="${camera_model}" />
     <xacro:property name="has_imu" value="false" />
-    <xacro:property name="is_bno" value="false"/>
     <!-- <xacro:if value="${model == 'BW1098OAK'}">
     </xacro:if> -->
@@ -20,24 +19,4 @@
       <xacro:property name="imu_p" value="1.5708" />
       <xacro:property name="imu_y" value="0" />
-    </xacro:if>
-    <xacro:if value="${model == 'OAK-D-PRO-W'}">
-      <xacro:if value="${is_bno}">
-        <xacro:property name="has_imu" value="true" />
-        <xacro:property name="imu_offset_x" value="0.075448" />
-        <xacro:property name="imu_offset_y" value="0.0079" />
-        <xacro:property name="imu_offset_z" value="0.0" />
-        <xacro:property name="imu_r" value="-3.1415" />
-        <xacro:property name="imu_p" value="0.0" />
-        <xacro:property name="imu_y" value="-1.5708" />
-      </xacro:if>
-      <xacro:unless value="${is_bno}">
-        <xacro:property name="has_imu" value="true" />
-        <xacro:property name="imu_offset_x" value="0.06935" />
-        <xacro:property name="imu_offset_y" value="0.00231" />
-        <xacro:property name="imu_offset_z" value="0.0" />
-        <xacro:property name="imu_r" value="-3.1415" />
-        <xacro:property name="imu_p" value="0.0" />
-        <xacro:property name="imu_y" value="-1.5708" />
-      </xacro:unless>
     </xacro:if>
     <!-- base_link of the sensor-->
