Commit message: add imu from description

File: depthai_descriptions/urdf/base_descr.urdf.xacro (robot description, xacro)
@@ -11,6 +11,7 @@
     <xacro:arg name="cam_pitch"     default="0.0" />
     <xacro:arg name="cam_yaw"       default="0.0" />
+    <xacro:arg name="has_imu"       default="false" />
     <xacro:include filename="$(find depthai_descriptions)/urdf/include/base_macro.urdf.xacro"/>
     <link name="$(arg parent_frame)"/>
-    <xacro:base camera_name = "$(arg camera_name)" parent = "$(arg parent_frame)" camera_model = "$(arg camera_model)" base_frame = "$(arg base_frame)" cam_pos_x = "$(arg cam_pos_x)" cam_pos_y = "$(arg cam_pos_y)" cam_pos_z = "$(arg cam_pos_z)" cam_roll = "$(arg cam_roll)" cam_pitch = "$(arg cam_pitch)" cam_yaw = "$(arg cam_yaw)"/>
+    <xacro:base camera_name = "$(arg camera_name)" parent = "$(arg parent_frame)" camera_model = "$(arg camera_model)" base_frame = "$(arg base_frame)" cam_pos_x = "$(arg cam_pos_x)" cam_pos_y = "$(arg cam_pos_y)" cam_pos_z = "$(arg cam_pos_z)" cam_roll = "$(arg cam_roll)" cam_pitch = "$(arg cam_pitch)" cam_yaw = "$(arg cam_yaw)" has_imu="$(arg has_imu)"/>
 </robot>

File: depthai_descriptions/urdf/include/base_macro.urdf.xacro (robot description, xacro)
@@ -4,5 +4,5 @@
     <xacro:macro name="base" params="camera_name camera_model parent base_frame
                                            cam_pos_x cam_pos_y cam_pos_z
-                                           cam_roll cam_pitch cam_yaw r:=0.8 g:=0.8 b:=0.8 a:=0.8">
+                                           cam_roll cam_pitch cam_yaw has_imu r:=0.8 g:=0.8 b:=0.8 a:=0.8 ">
         <!-- base_link of the sensor-->
         <link name="${base_frame}"/>
@@ -31,4 +31,21 @@
             <origin xyz="0 0 0" rpy="1.5708 0 1.5708" />
         </joint>
+        <!-- IMU -->
+        <xacro:if value="${model == 'OAK-D'}">
+            <xacro:property name="imu_offset_x" value="0.0" />
+            <xacro:property name="imu_offset_y" value="-0.015" />
+            <xacro:property name="imu_offset_z" value="-0.013662" />
+            <xacro:property name="imu_r" value="0" />
+            <xacro:property name="imu_p" value="1.5708" />
+            <xacro:property name="imu_y" value="0" />
+        </xacro:if>
+        <xacro:if value="${has_imu}">
+            <link name="${camera_name}_imu_frame" />
+            <joint name="${camera_name}_imu_joint" type="fixed">
+                <parent link="${base_frame}"/>
+                <child link="${camera_name}_imu_frame"/>
+                <origin xyz="${imu_offset_x} ${imu_offset_y} ${imu_offset_z}" rpy="${imu_r} ${imu_p} ${imu_y}" />
+            </joint>
+        </xacro:if>
     </xacro:macro>
 </robot>

File: depthai_descriptions/urdf/include/depthai_macro.urdf.xacro (robot description, xacro)
@@ -9,26 +9,9 @@
         <xacro:property name="model" value="${camera_model}" />
         <xacro:property name="has_imu" value="false" />
-        <!-- <xacro:if value="${model == 'BW1098OAK'}">
-    </xacro:if> -->
         <xacro:property name="baseline" value="0.075" />
         <xacro:if value="${model == 'OAK-D'}">
             <xacro:property name="has_imu" value="true" />
-            <xacro:property name="imu_offset_x" value="0.0" />
-            <xacro:property name="imu_offset_y" value="-0.015" />
-            <xacro:property name="imu_offset_z" value="-0.013662" />
-            <xacro:property name="imu_r" value="0" />
-            <xacro:property name="imu_p" value="1.5708" />
-            <xacro:property name="imu_y" value="0" />
         </xacro:if>
-        <xacro:base camera_name = "$(arg camera_name)" parent = "$(arg parent_frame)" camera_model = "$(arg camera_model)" base_frame = "$(arg base_frame)" cam_pos_x = "$(arg cam_pos_x)" cam_pos_y = "$(arg cam_pos_y)" cam_pos_z = "$(arg cam_pos_z)" cam_roll = "$(arg cam_roll)" cam_pitch = "$(arg cam_pitch)" cam_yaw = "$(arg cam_yaw)"/>
-        <!-- IMU -->
-        <xacro:if value="${has_imu}">
-            <link name="${camera_name}_imu_frame" />
-            <joint name="${camera_name}_imu_joint" type="fixed">
-                <parent link="${base_frame}"/>
-                <child link="${camera_name}_imu_frame"/>
-                <origin xyz="${imu_offset_x} ${imu_offset_y} ${imu_offset_z}" rpy="${imu_r} ${imu_p} ${imu_y}" />
-            </joint>
-        </xacro:if>
+        <xacro:base camera_name = "$(arg camera_name)" parent = "$(arg parent_frame)" camera_model = "$(arg camera_model)" base_frame = "$(arg base_frame)" cam_pos_x = "$(arg cam_pos_x)" cam_pos_y = "$(arg cam_pos_y)" cam_pos_z = "$(arg cam_pos_z)" cam_roll = "$(arg cam_roll)" cam_pitch = "$(arg cam_pitch)" cam_yaw = "$(arg cam_yaw)" has_imu="${has_imu}"/>
         <!-- RGB Camera -->
         <link name="${camera_name}_rgb_camera_frame" />
