Commit message: Add missing descriptions

File: depthai_descriptions/urdf/base_descr.urdf.xacro (robot description, xacro)
@@ -2,4 +2,6 @@
 <robot name="depthai_camera" xmlns:xacro="http://ros.org/wiki/xacro">
 	<xacro:arg name="camera_name" default="oak" />
+	<xacro:arg name="imu_sensor" default="" />
+	<xacro:arg name="imu_frame" default="optical" />
 	<xacro:arg name="camera_model" default="OAK-D" />
 	<xacro:arg name="base_frame" default="oak" />
@@ -15,5 +17,5 @@
 	<link name="$(arg parent_frame)" />
 	<xacro:base camera_name="$(arg camera_name)" parent="$(arg parent_frame)"
-		camera_model="$(arg camera_model)" base_frame="$(arg base_frame)"
+		camera_model="$(arg camera_model)" imu_sensor="$(arg imu_sensor)" imu_frame="$(arg imu_frame)" base_frame="$(arg base_frame)"
 		cam_pos_x="$(arg cam_pos_x)" cam_pos_y="$(arg cam_pos_y)" cam_pos_z="$(arg cam_pos_z)"
 		cam_roll="$(arg cam_roll)" cam_pitch="$(arg cam_pitch)" cam_yaw="$(arg cam_yaw)"

File: depthai_descriptions/urdf/depthai_descr.urdf.xacro (robot description, xacro)
@@ -2,4 +2,6 @@
 <robot name="depthai_camera" xmlns:xacro="http://ros.org/wiki/xacro">
 	<xacro:arg name="camera_name" default="oak" />
+	<xacro:arg name="imu_sensor" default="" />
+	<xacro:arg name="imu_frame" default="optical" />
 	<xacro:arg name="camera_model" default="OAK-D" />
 	<xacro:arg name="base_frame" default="oak" />
@@ -15,5 +17,5 @@
 	<link name="$(arg parent_frame)" />
 	<xacro:depthai_camera camera_name="$(arg camera_name)" parent="$(arg parent_frame)"
-		camera_model="$(arg camera_model)" base_frame="$(arg base_frame)"
+		camera_model="$(arg camera_model)" imu_sensor="$(arg imu_sensor)" imu_frame="$(arg imu_frame)" base_frame="$(arg base_frame)"
 		cam_pos_x="$(arg cam_pos_x)" cam_pos_y="$(arg cam_pos_y)" cam_pos_z="$(arg cam_pos_z)"
 		cam_roll="$(arg cam_roll)" cam_pitch="$(arg cam_pitch)" cam_yaw="$(arg cam_yaw)"

File: depthai_descriptions/urdf/include/base_macro.urdf.xacro (robot description, xacro)
@@ -6,6 +6,6 @@
 		params="camera_name camera_model parent base_frame
                                            cam_pos_x cam_pos_y cam_pos_z
-                                           cam_roll cam_pitch cam_yaw has_imu r:=0.8 g:=0.8 b:=0.8 a:=0.8 simulation:=false">
-		<xacro:depthai_model_config camera_model="${camera_model}" />
+                                           cam_roll cam_pitch cam_yaw has_imu r:=0.8 g:=0.8 b:=0.8 a:=0.8 simulation:=false imu_sensor:='' imu_frame:='optical'">
+		<xacro:depthai_model_config camera_model="${camera_model}" imu_sensor="${imu_sensor}" imu_frame="${imu_frame}" />
 		<xacro:if value="${simulation}">
 			<xacro:property
@@ -31,13 +31,15 @@
 		<!-- device Center -->
 		<link name="${camera_name}_model_origin">
-			<visual>
-				<origin xyz="${device_config['mesh_xyz']}" rpy="0 0 0" />
-				<geometry>
-					<mesh filename="${file_prefix}/urdf/models/${model}.stl" />
-				</geometry>
-				<material name="mat">
-					<color rgba="${r} ${g} ${b} ${a}" />
-				</material>
-			</visual>
+			<xacro:if value="${device_config['mesh'] is not None}">
+				<visual>
+					<origin xyz="${device_config['mesh_xyz']}" rpy="0 0 0" />
+					<geometry>
+						<mesh filename="${file_prefix}/urdf/models/${device_config['mesh']}.stl" />
+					</geometry>
+					<material name="mat">
+						<color rgba="${r} ${g} ${b} ${a}" />
+					</material>
+				</visual>
+			</xacro:if>
 		</link>
 		<joint name="${camera_name}_model_origin_joint" type="fixed">
@@ -50,5 +52,5 @@
 			<xacro:if value="${device_config['imu_xyz'] is None or device_config['imu_rpy'] is None}">
 				<xacro:property name="invalid_imu" lazy_eval="false"
-					value="${xacro.fatal('No IMU transform defined for camera_model: ' + camera_model)}" />
+					value="${xacro.fatal('No selected IMU transform for ' + camera_model + '. Set imu_sensor to one of: ' + ', '.join(device_config['imu_variants'].keys()))}" />
 			</xacro:if>
 			<link name="${camera_name}_imu_frame" />

File: depthai_descriptions/urdf/include/depthai_macro.urdf.xacro (robot description, xacro)
@@ -4,5 +4,5 @@
 	<!-- Camera and optical frames share the same structure for every sensor. -->
 	<xacro:macro name="depthai_camera_frame"
-		params="camera_name base_frame sensor_name joint_name xyz frame_suffix optical_frame_suffix">
+		params="camera_name base_frame sensor_name joint_name xyz frame_suffix optical_frame_suffix rpy:='0 0 0'">
 		<xacro:property name="M_PI" value="3.1415926535897931" />
 		<link name="${camera_name}_${sensor_name}_${frame_suffix}" />
@@ -10,5 +10,5 @@
 			<parent link="${base_frame}" />
 			<child link="${camera_name}_${sensor_name}_${frame_suffix}" />
-			<origin xyz="${xyz}" rpy="0 0 0" />
+			<origin xyz="${xyz}" rpy="${rpy}" />
 		</joint>
 		<link name="${camera_name}_${sensor_name}_${optical_frame_suffix}" />
@@ -19,10 +19,21 @@
 		</joint>
 	</xacro:macro>
+	<!-- Recursive expansion preserves extra sockets on boards with >3 cameras. -->
+	<xacro:macro name="depthai_extra_cameras" params="names cameras camera_name base_frame frame_suffix optical_frame_suffix">
+		<xacro:if value="${len(names) > 0}">
+			<xacro:property name="sensor" value="${names[0]}" />
+			<xacro:depthai_camera_frame camera_name="${camera_name}" base_frame="${base_frame}"
+				sensor_name="${sensor}" joint_name="${sensor}" xyz="${cameras[sensor]['xyz']}"
+				rpy="${cameras[sensor]['rpy']}" frame_suffix="${frame_suffix}" optical_frame_suffix="${optical_frame_suffix}" />
+			<xacro:depthai_extra_cameras names="${names[1:]}" cameras="${cameras}" camera_name="${camera_name}"
+				base_frame="${base_frame}" frame_suffix="${frame_suffix}" optical_frame_suffix="${optical_frame_suffix}" />
+		</xacro:if>
+	</xacro:macro>
 	<xacro:macro name="depthai_camera"
 		params="camera_name camera_model parent base_frame
                                            cam_pos_x cam_pos_y cam_pos_z
-                                           cam_roll cam_pitch cam_yaw r:=0.8 g:=0.8 b:=0.8 a:=0.8 simulation:=false rs_compat:=false">
+                                           cam_roll cam_pitch cam_yaw r:=0.8 g:=0.8 b:=0.8 a:=0.8 simulation:=false rs_compat:=false imu_sensor:='' imu_frame:='optical'">
 		<xacro:include filename="$(find depthai_descriptions)/urdf/include/base_macro.urdf.xacro" />
-		<xacro:depthai_model_config camera_model="${camera_model}" />
+		<xacro:depthai_model_config camera_model="${camera_model}" imu_sensor="${imu_sensor}" imu_frame="${imu_frame}" />
 		<xacro:if value="${rs_compat}">
 			<xacro:property name="frame_suffix" value="frame" />
@@ -42,20 +53,23 @@
 			base_frame="${base_frame}" cam_pos_x="${cam_pos_x}" cam_pos_y="${cam_pos_y}"
 			cam_pos_z="${cam_pos_z}" cam_roll="${cam_roll}" cam_pitch="${cam_pitch}"
-			cam_yaw="${cam_yaw}" has_imu="${device_config['imu_xyz'] is not None}" simulation="${simulation}" />
+			cam_yaw="${cam_yaw}" has_imu="${device_config['imu_xyz'] is not None}" simulation="${simulation}" imu_sensor="${imu_sensor}" imu_frame="${imu_frame}" />
 		<xacro:if value="${device_config['rgb_xyz'] is not None}">
 			<xacro:depthai_camera_frame camera_name="${camera_name}" base_frame="${base_frame}"
-				sensor_name="${rgb_name}" joint_name="rgb" xyz="${device_config['rgb_xyz']}"
+				sensor_name="${rgb_name}" joint_name="rgb" xyz="${device_config['rgb_xyz']}" rpy="${device_config['rgb_rpy']}"
 				frame_suffix="${frame_suffix}" optical_frame_suffix="${optical_frame_suffix}" />
 		</xacro:if>
 		<xacro:if value="${device_config['left_xyz'] is not None}">
 			<xacro:depthai_camera_frame camera_name="${camera_name}" base_frame="${base_frame}"
-				sensor_name="${left_name}" joint_name="left" xyz="${device_config['left_xyz']}"
+				sensor_name="${left_name}" joint_name="left" xyz="${device_config['left_xyz']}" rpy="${device_config['left_rpy']}"
 				frame_suffix="${frame_suffix}" optical_frame_suffix="${optical_frame_suffix}" />
 		</xacro:if>
 		<xacro:if value="${device_config['right_xyz'] is not None}">
 			<xacro:depthai_camera_frame camera_name="${camera_name}" base_frame="${base_frame}"
-				sensor_name="${device_config['right_name'] or right_name}" joint_name="right" xyz="${device_config['right_xyz']}"
+				sensor_name="${device_config['right_name'] or right_name}" joint_name="right" xyz="${device_config['right_xyz']}" rpy="${device_config['right_rpy']}"
 				frame_suffix="${frame_suffix}" optical_frame_suffix="${optical_frame_suffix}" />
 		</xacro:if>
+		<xacro:depthai_extra_cameras names="${list(device_config['extra_cameras'].keys())}"
+			cameras="${device_config['extra_cameras']}" camera_name="${camera_name}" base_frame="${base_frame}"
+			frame_suffix="${frame_suffix}" optical_frame_suffix="${optical_frame_suffix}" />
 	</xacro:macro>
 </robot>

File: depthai_descriptions/urdf/include/model_config.urdf.xacro (robot description, xacro)
@@ -2,9 +2,25 @@
 <robot xmlns:xacro="http://ros.org/wiki/xacro">
 	<!-- Export a fresh configuration into the calling macro's scope. -->
-	<xacro:macro name="depthai_model_config" params="camera_model">
+	<xacro:macro name="depthai_model_config" params="camera_model imu_sensor:='' imu_frame:='optical'">
 		<xacro:property name="config_file" value="$(find depthai_descriptions)/urdf/include/model_config.yaml" />
 		<xacro:property name="configs" value="${xacro.load_yaml(config_file)}" />
+		<xacro:property name="boards" value="${xacro.load_yaml('$(find depthai_descriptions)/urdf/include/board_models.yaml')}" />
+		<xacro:if value="${camera_model in boards['unsupported']}">
+			<xacro:property name="invalid_board" lazy_eval="false"
+				value="${xacro.fatal('Cannot place board ' + camera_model + ': ' + boards['unsupported'][camera_model])}" />
+		</xacro:if>
+		<xacro:property name="overrides" value="${configs['models'].get(camera_model, dict())}" />
+		<xacro:property name="board_config" value="${boards['models'].get(camera_model, dict(mesh=camera_model))}" />
+		<xacro:property name="merged" value="${dict(dict(configs['defaults'], **board_config), **overrides)}" />
+		<xacro:property name="variants" value="${merged['imu_variants']}" />
+		<xacro:if value="${imu_frame not in ['native', 'optical'] or (imu_sensor != '' and imu_sensor not in variants)}">
+			<xacro:property name="invalid_imu_selection" lazy_eval="false"
+				value="${xacro.fatal('Invalid IMU selection for ' + camera_model + ': sensor=' + imu_sensor + ', frame=' + imu_frame + '; available sensors: ' + ', '.join(variants.keys()))}" />
+		</xacro:if>
+		<xacro:property name="selected" value="${imu_sensor if imu_sensor != '' else (list(variants.keys())[0] if len(variants) == 1 else '')}" />
+		<xacro:property name="use_board_imu" value="${selected != '' and (imu_sensor != '' or overrides.get('imu_xyz') is None)}" />
+		<xacro:property name="imu_override" value="${dict(imu_xyz=variants[selected]['xyz'], imu_rpy=variants[selected][imu_frame + '_rpy']) if use_board_imu else dict()}" />
 		<xacro:property name="device_config" scope="parent"
-			value="${dict(configs['defaults'], **configs['models'].get(camera_model, dict()))}" />
+			value="${dict(merged, **imu_override)}" />
 	</xacro:macro>
 </robot>
