Commit message: Integrate board URDFs while preserving legacy compatibility

File: depthai_descriptions/urdf/base_descr.urdf.xacro (robot description, xacro)
@@ -3,5 +3,7 @@
 	<xacro:arg name="camera_name" default="oak" />
 	<xacro:arg name="imu_sensor" default="" />
-	<xacro:arg name="imu_frame" default="optical" />
+	<xacro:arg name="imu_frame" default="auto" />
+	<xacro:arg name="pose_source" default="legacy" />
+	<xacro:arg name="mesh_model" default="" />
 	<xacro:arg name="camera_model" default="OAK-D" />
 	<xacro:arg name="base_frame" default="oak" />
@@ -17,5 +19,5 @@
 	<link name="$(arg parent_frame)" />
 	<xacro:base camera_name="$(arg camera_name)" parent="$(arg parent_frame)"
-		camera_model="$(arg camera_model)" imu_sensor="$(arg imu_sensor)" imu_frame="$(arg imu_frame)" base_frame="$(arg base_frame)"
+		camera_model="$(arg camera_model)" imu_sensor="$(arg imu_sensor)" imu_frame="$(arg imu_frame)" pose_source="$(arg pose_source)" mesh_model="$(arg mesh_model)" base_frame="$(arg base_frame)"
 		cam_pos_x="$(arg cam_pos_x)" cam_pos_y="$(arg cam_pos_y)" cam_pos_z="$(arg cam_pos_z)"
 		cam_roll="$(arg cam_roll)" cam_pitch="$(arg cam_pitch)" cam_yaw="$(arg cam_yaw)"

File: depthai_descriptions/urdf/depthai_descr.urdf.xacro (robot description, xacro)
@@ -2,6 +2,10 @@
 <robot name="depthai_camera" xmlns:xacro="http://ros.org/wiki/xacro">
 	<xacro:arg name="camera_name" default="oak" />
+	<xacro:arg name="has_imu" default="auto" />
 	<xacro:arg name="imu_sensor" default="" />
-	<xacro:arg name="imu_frame" default="optical" />
+	<xacro:arg name="imu_frame" default="auto" />
+	<xacro:arg name="legacy_frame_aliases" default="true" />
+	<xacro:arg name="pose_source" default="legacy" />
+	<xacro:arg name="mesh_model" default="" />
 	<xacro:arg name="camera_model" default="OAK-D" />
 	<xacro:arg name="base_frame" default="oak" />
@@ -17,7 +21,7 @@
 	<link name="$(arg parent_frame)" />
 	<xacro:depthai_camera camera_name="$(arg camera_name)" parent="$(arg parent_frame)"
-		camera_model="$(arg camera_model)" imu_sensor="$(arg imu_sensor)" imu_frame="$(arg imu_frame)" base_frame="$(arg base_frame)"
+		camera_model="$(arg camera_model)" imu_sensor="$(arg imu_sensor)" imu_frame="$(arg imu_frame)" pose_source="$(arg pose_source)" mesh_model="$(arg mesh_model)" base_frame="$(arg base_frame)"
 		cam_pos_x="$(arg cam_pos_x)" cam_pos_y="$(arg cam_pos_y)" cam_pos_z="$(arg cam_pos_z)"
 		cam_roll="$(arg cam_roll)" cam_pitch="$(arg cam_pitch)" cam_yaw="$(arg cam_yaw)"
-		rs_compat="$(arg rs_compat)" />
+		rs_compat="$(arg rs_compat)" legacy_frame_aliases="$(arg legacy_frame_aliases)" has_imu="$(arg has_imu)" />
 </robot>

File: depthai_descriptions/urdf/include/base_macro.urdf.xacro (robot description, xacro)
@@ -6,6 +6,11 @@
 		params="camera_name camera_model parent base_frame
                                            cam_pos_x cam_pos_y cam_pos_z
-                                           cam_roll cam_pitch cam_yaw has_imu r:=0.8 g:=0.8 b:=0.8 a:=0.8 simulation:=false imu_sensor:='' imu_frame:='optical'">
-		<xacro:depthai_model_config camera_model="${camera_model}" imu_sensor="${imu_sensor}" imu_frame="${imu_frame}" />
+                                           cam_roll cam_pitch cam_yaw has_imu r:=0.8 g:=0.8 b:=0.8 a:=0.8 simulation:=false imu_sensor:='' imu_frame:='auto' pose_source:='legacy' mesh_model:=''">
+		<xacro:depthai_model_config camera_model="${camera_model}" imu_sensor="${imu_sensor}" imu_frame="${imu_frame}" pose_source="${pose_source}" mesh_model="${mesh_model}" />
+        <!-- Warn here once per device, including direct Xacro/macro users. -->
+        <xacro:if value="${device_config['legacy']}">
+            <xacro:property name="legacy_pose_warning" lazy_eval="false"
+                value="${xacro.warning('DEPRECATED pose_source=legacy: using frozen develop geometry for ' + camera_model + '. ' + ('No depthai_boards counterpart is available for this model.' if camera_model == 'OAK-D-IOT-75' else 'Select pose_source:=board to use depthai_boards geometry.'))}" />
+        </xacro:if>
 		<xacro:if value="${simulation}">
 			<xacro:property
@@ -46,5 +51,5 @@
 			<parent link="${base_frame}" />
 			<child link="${camera_name}_model_origin" />
-			<origin xyz="0 0 0" rpy="1.5708 0 1.5708" />
+			<origin xyz="${device_config['mesh_base_xyz']}" rpy="1.5708 0 1.5708" />
 		</joint>
 		<!-- IMU -->

File: depthai_descriptions/urdf/include/depthai_macro.urdf.xacro (robot description, xacro)
@@ -2,7 +2,17 @@
 <robot name="depthai_camera"
 	xmlns:xacro="http://ros.org/wiki/xacro">
+    <!-- DEPRECATED identity aliases: migrate consumers to the socket-based names. -->
+    <xacro:macro name="depthai_frame_alias" params="canonical alias">
+        <xacro:if value="${canonical != alias}">
+            <link name="${alias}" />
+            <joint name="${alias}_deprecated_alias_joint" type="fixed">
+                <parent link="${canonical}" /><child link="${alias}" />
+                <origin xyz="0 0 0" rpy="0 0 0" />
+            </joint>
+        </xacro:if>
+    </xacro:macro>
 	<!-- Camera and optical frames share the same structure for every sensor. -->
 	<xacro:macro name="depthai_camera_frame"
-		params="camera_name base_frame sensor_name joint_name xyz frame_suffix optical_frame_suffix rpy:='0 0 0'">
+		params="camera_name base_frame sensor_name joint_name xyz frame_suffix optical_frame_suffix rpy:='0 0 0' legacy_name:='' aliases:=false reserved_names:=''">
 		<xacro:property name="M_PI" value="3.1415926535897931" />
 		<link name="${camera_name}_${sensor_name}_${frame_suffix}" />
@@ -18,13 +28,23 @@
 			<child link="${camera_name}_${sensor_name}_${optical_frame_suffix}" />
 		</joint>
-	</xacro:macro>
-	<!-- Recursive expansion preserves extra sockets on boards with >3 cameras. -->
-	<xacro:macro name="depthai_extra_cameras" params="names cameras camera_name base_frame frame_suffix optical_frame_suffix">
+        <xacro:if value="${aliases}">
+            <xacro:depthai_frame_alias canonical="${camera_name}_${sensor_name}_${frame_suffix}" alias="${camera_name}_${sensor_name}_camera_frame" />
+            <xacro:if value="${legacy_name != '' and legacy_name != sensor_name and legacy_name not in reserved_names}">
+                <xacro:depthai_frame_alias canonical="${camera_name}_${sensor_name}_${frame_suffix}" alias="${camera_name}_${legacy_name}_camera_frame" />
+                <xacro:depthai_frame_alias canonical="${camera_name}_${sensor_name}_${optical_frame_suffix}" alias="${camera_name}_${legacy_name}_${optical_frame_suffix}" />
+                <xacro:if value="${frame_suffix == 'frame'}">
+                    <xacro:depthai_frame_alias canonical="${camera_name}_${sensor_name}_${frame_suffix}" alias="${camera_name}_${legacy_name}_frame" />
+                </xacro:if>
+            </xacro:if>
+        </xacro:if>
+    </xacro:macro>
+    <!-- Recursive expansion preserves extra sockets on boards with >3 cameras. -->
+	<xacro:macro name="depthai_extra_cameras" params="names cameras camera_name base_frame frame_suffix optical_frame_suffix socket_names aliases">
 		<xacro:if value="${len(names) > 0}">
 			<xacro:property name="sensor" value="${names[0]}" />
 			<xacro:depthai_camera_frame camera_name="${camera_name}" base_frame="${base_frame}"
-				sensor_name="${sensor}" joint_name="${sensor}" xyz="${cameras[sensor]['xyz']}"
-				rpy="${cameras[sensor]['rpy']}" frame_suffix="${frame_suffix}" optical_frame_suffix="${optical_frame_suffix}" />
-			<xacro:depthai_extra_cameras names="${names[1:]}" cameras="${cameras}" camera_name="${camera_name}"
+				sensor_name="${socket_names.get(cameras[sensor]['socket'], sensor)}" joint_name="${sensor}" xyz="${cameras[sensor]['xyz']}"
+				rpy="${cameras[sensor]['rpy']}" aliases="${aliases}" legacy_name="${sensor}" reserved_names="${list(socket_names.values())}" frame_suffix="${frame_suffix}" optical_frame_suffix="${optical_frame_suffix}" />
+			<xacro:depthai_extra_cameras names="${names[1:]}" aliases="${aliases}" cameras="${cameras}" socket_names="${socket_names}" camera_name="${camera_name}"
 				base_frame="${base_frame}" frame_suffix="${frame_suffix}" optical_frame_suffix="${optical_frame_suffix}" />
 		</xacro:if>
@@ -33,7 +53,7 @@
 		params="camera_name camera_model parent base_frame
                                            cam_pos_x cam_pos_y cam_pos_z
-                                           cam_roll cam_pitch cam_yaw r:=0.8 g:=0.8 b:=0.8 a:=0.8 simulation:=false rs_compat:=false imu_sensor:='' imu_frame:='optical'">
+                                           cam_roll cam_pitch cam_yaw r:=0.8 g:=0.8 b:=0.8 a:=0.8 simulation:=false rs_compat:=false has_imu:='auto' imu_sensor:='' imu_frame:='auto' pose_source:='legacy' mesh_model:='' legacy_frame_aliases:=true">
 		<xacro:include filename="$(find depthai_descriptions)/urdf/include/base_macro.urdf.xacro" />
-		<xacro:depthai_model_config camera_model="${camera_model}" imu_sensor="${imu_sensor}" imu_frame="${imu_frame}" />
+		<xacro:depthai_model_config camera_model="${camera_model}" imu_sensor="${imu_sensor}" imu_frame="${imu_frame}" pose_source="${pose_source}" mesh_model="${mesh_model}" />
 		<xacro:if value="${rs_compat}">
 			<xacro:property name="frame_suffix" value="frame" />
@@ -50,25 +70,33 @@
 			<xacro:property name="right_name" value="right" />
 		</xacro:unless>
+		<!-- Keep names identical to depthai_bridge::getSocketName in both TF modes. -->
+		<xacro:property name="socket_names" value="${dict(CAM_A=rgb_name, CAM_B=left_name, CAM_C=right_name, CAM_D=('infra3' if rs_compat else 'left_back'), CAM_E=('infra4' if rs_compat else 'right_back'))}" />
+		<xacro:if value="${camera_model == 'OAK-D-SR-POE'}">
+			<xacro:property name="socket_names" value="${dict(CAM_A='tof', CAM_B='left', CAM_C='right')}" />
+		</xacro:if>
+		<xacro:if value="${camera_model == 'OAK-T'}">
+			<xacro:property name="socket_names" value="${dict(CAM_A='rgb', CAM_B='left', CAM_C='right', CAM_D='left_back', CAM_E='thermal')}" />
+		</xacro:if>
 		<xacro:base camera_name="${camera_name}" parent="${parent}" camera_model="${camera_model}"
 			base_frame="${base_frame}" cam_pos_x="${cam_pos_x}" cam_pos_y="${cam_pos_y}"
 			cam_pos_z="${cam_pos_z}" cam_roll="${cam_roll}" cam_pitch="${cam_pitch}"
-			cam_yaw="${cam_yaw}" has_imu="${device_config['imu_xyz'] is not None}" simulation="${simulation}" imu_sensor="${imu_sensor}" imu_frame="${imu_frame}" />
+			cam_yaw="${cam_yaw}" has_imu="${device_config['imu_xyz'] is not None if has_imu == 'auto' else has_imu}" simulation="${simulation}" imu_sensor="${imu_sensor}" imu_frame="${imu_frame}" pose_source="${pose_source}" mesh_model="${mesh_model}" />
 		<xacro:if value="${device_config['rgb_xyz'] is not None}">
 			<xacro:depthai_camera_frame camera_name="${camera_name}" base_frame="${base_frame}"
-				sensor_name="${rgb_name}" joint_name="rgb" xyz="${device_config['rgb_xyz']}" rpy="${device_config['rgb_rpy']}"
+				sensor_name="${socket_names.get(device_config.get('rgb_socket'), rgb_name)}" joint_name="rgb" aliases="${legacy_frame_aliases and not device_config['legacy']}" legacy_name="${rgb_name}" reserved_names="${list(socket_names.values())}" xyz="${device_config['rgb_xyz']}" rpy="${device_config['rgb_rpy']}"
 				frame_suffix="${frame_suffix}" optical_frame_suffix="${optical_frame_suffix}" />
 		</xacro:if>
 		<xacro:if value="${device_config['left_xyz'] is not None}">
 			<xacro:depthai_camera_frame camera_name="${camera_name}" base_frame="${base_frame}"
-				sensor_name="${left_name}" joint_name="left" xyz="${device_config['left_xyz']}" rpy="${device_config['left_rpy']}"
+				sensor_name="${socket_names.get(device_config.get('left_socket'), left_name)}" joint_name="left" aliases="${legacy_frame_aliases and not device_config['legacy']}" legacy_name="${left_name}" reserved_names="${list(socket_names.values())}" xyz="${device_config['left_xyz']}" rpy="${device_config['left_rpy']}"
 				frame_suffix="${frame_suffix}" optical_frame_suffix="${optical_frame_suffix}" />
 		</xacro:if>
 		<xacro:if value="${device_config['right_xyz'] is not None}">
 			<xacro:depthai_camera_frame camera_name="${camera_name}" base_frame="${base_frame}"
-				sensor_name="${device_config['right_name'] or right_name}" joint_name="right" xyz="${device_config['right_xyz']}" rpy="${device_config['right_rpy']}"
+				sensor_name="${device_config['right_name'] or socket_names.get(device_config.get('right_socket'), right_name)}" joint_name="right" aliases="${legacy_frame_aliases and not device_config['legacy']}" legacy_name="${'cam_e' if camera_model == 'OAK-T' else right_name}" reserved_names="${list(socket_names.values())}" xyz="${device_config['right_xyz']}" rpy="${device_config['right_rpy']}"
 				frame_suffix="${frame_suffix}" optical_frame_suffix="${optical_frame_suffix}" />
 		</xacro:if>
 		<xacro:depthai_extra_cameras names="${list(device_config['extra_cameras'].keys())}"
-			cameras="${device_config['extra_cameras']}" camera_name="${camera_name}" base_frame="${base_frame}"
+			cameras="${device_config['extra_cameras']}" aliases="${legacy_frame_aliases and not device_config['legacy']}" socket_names="${socket_names}" camera_name="${camera_name}" base_frame="${base_frame}"
 			frame_suffix="${frame_suffix}" optical_frame_suffix="${optical_frame_suffix}" />
 	</xacro:macro>

File: depthai_descriptions/urdf/include/model_config.urdf.xacro (robot description, xacro)
@@ -1,26 +1,28 @@
 <?xml version="1.0"?>
 <robot xmlns:xacro="http://ros.org/wiki/xacro">
-	<!-- Export a fresh configuration into the calling macro's scope. -->
-	<xacro:macro name="depthai_model_config" params="camera_model imu_sensor:='' imu_frame:='optical'">
-		<xacro:property name="config_file" value="$(find depthai_descriptions)/urdf/include/model_config.yaml" />
-		<xacro:property name="configs" value="${xacro.load_yaml(config_file)}" />
-		<xacro:property name="boards" value="${xacro.load_yaml('$(find depthai_descriptions)/urdf/include/board_models.yaml')}" />
-		<xacro:if value="${camera_model in boards['unsupported']}">
-			<xacro:property name="invalid_board" lazy_eval="false"
-				value="${xacro.fatal('Cannot place board ' + camera_model + ': ' + boards['unsupported'][camera_model])}" />
-		</xacro:if>
-		<xacro:property name="overrides" value="${configs['models'].get(camera_model, dict())}" />
-		<xacro:property name="board_config" value="${boards['models'].get(camera_model, dict(mesh=camera_model))}" />
-		<xacro:property name="merged" value="${dict(dict(configs['defaults'], **board_config), **overrides)}" />
-		<xacro:property name="variants" value="${merged['imu_variants']}" />
-		<xacro:if value="${imu_frame not in ['native', 'optical'] or (imu_sensor != '' and imu_sensor not in variants)}">
-			<xacro:property name="invalid_imu_selection" lazy_eval="false"
-				value="${xacro.fatal('Invalid IMU selection for ' + camera_model + ': sensor=' + imu_sensor + ', frame=' + imu_frame + '; available sensors: ' + ', '.join(variants.keys()))}" />
-		</xacro:if>
-		<xacro:property name="selected" value="${imu_sensor if imu_sensor != '' else (list(variants.keys())[0] if len(variants) == 1 else '')}" />
-		<xacro:property name="use_board_imu" value="${selected != '' and (imu_sensor != '' or overrides.get('imu_xyz') is None)}" />
-		<xacro:property name="imu_override" value="${dict(imu_xyz=variants[selected]['xyz'], imu_rpy=variants[selected][imu_frame + '_rpy']) if use_board_imu else dict()}" />
-		<xacro:property name="device_config" scope="parent"
-			value="${dict(merged, **imu_override)}" />
-	</xacro:macro>
+  <xacro:macro name="depthai_model_config" params="camera_model imu_sensor:='' imu_frame:='auto' pose_source:='legacy' mesh_model:=''">
+    <xacro:property name="configs" value="${xacro.load_yaml('$(find depthai_descriptions)/urdf/include/model_config.yaml')}" />
+    <xacro:property name="boards" value="${xacro.load_yaml('$(find depthai_descriptions)/urdf/include/board_models.yaml')}" />
+    <!-- DEPRECATED: frozen develop poses preserve existing installations. Opt into pose_source=board. -->
+    <xacro:property name="legacy" value="${xacro.load_yaml('$(find depthai_descriptions)/urdf/include/legacy_models.yaml')['models']}" />
+    <xacro:property name="resolved_model" value="${camera_model if camera_model in boards['models'] or camera_model in legacy else configs.get('aliases', dict()).get(camera_model, camera_model)}" />
+    <xacro:if value="${pose_source not in ['legacy', 'board'] or imu_frame not in ['auto', 'native', 'optical']}">
+      <xacro:property name="invalid" lazy_eval="false" value="${xacro.fatal('Invalid pose_source or imu_frame')}" />
+    </xacro:if>
+    <xacro:property name="use_legacy" value="${pose_source == 'legacy' and resolved_model in legacy}" />
+    <xacro:if value="${not use_legacy and resolved_model not in boards['models']}">
+      <xacro:property name="invalid" lazy_eval="false" value="${xacro.fatal('No valid board description: ' + resolved_model)}" />
+    </xacro:if>
+    <xacro:property name="record" value="${legacy[resolved_model] if use_legacy else dict(boards['models'][resolved_model], **configs['models'].get(resolved_model, dict()))}" />
+    <xacro:property name="merged" value="${dict(configs['defaults'], **record)}" />
+    <xacro:property name="variants" value="${merged['imu_variants']}" />
+    <xacro:if value="${not use_legacy and imu_sensor != '' and imu_sensor not in variants}">
+      <xacro:property name="invalid" lazy_eval="false" value="${xacro.fatal('Invalid IMU selection: ' + imu_sensor)}" />
+    </xacro:if>
+    <xacro:property name="selected" value="${'' if use_legacy else (imu_sensor if imu_sensor != '' else (list(variants.keys())[0] if len(variants) == 1 else ''))}" />
+    <xacro:property name="mode" value="${'native' if imu_frame == 'auto' else imu_frame}" />
+    <xacro:property name="imu_override" value="${dict(imu_xyz=variants[selected]['xyz'], imu_rpy=variants[selected][mode + '_rpy']) if selected != '' else dict()}" />
+    <xacro:property name="mesh" value="${mesh_model if mesh_model != '' else (merged['mesh'] or configs.get('mesh_aliases', dict()).get(resolved_model))}" />
+    <xacro:property name="device_config" scope="parent" value="${dict(dict(merged, **imu_override), mesh=mesh, legacy=use_legacy)}" />
+  </xacro:macro>
 </robot>
