Commit message: modified IMU position

File: depthai_descriptions/urdf/include/depthai_macro.urdf.xacro (robot description, xacro)
@@ -24,19 +24,19 @@
       <xacro:if value="${is_bno}">
         <xacro:property name="has_imu" value="true" />
-        <xacro:property name="imu_offset_x" value="0.075448" />
+        <xacro:property name="imu_offset_x" value="0.000448" />
         <xacro:property name="imu_offset_y" value="0.0079" />
         <xacro:property name="imu_offset_z" value="0.0" />
         <xacro:property name="imu_r" value="-3.1415" />
         <xacro:property name="imu_p" value="0.0" />
-        <xacro:property name="imu_y" value="-1.5708" />
+        <xacro:property name="imu_y" value="1.5708" />
       </xacro:if>
       <xacro:unless value="${is_bno}">
         <xacro:property name="has_imu" value="true" />
-        <xacro:property name="imu_offset_x" value="0.06935" />
+        <xacro:property name="imu_offset_x" value="-0.00535" />
         <xacro:property name="imu_offset_y" value="0.00231" />
         <xacro:property name="imu_offset_z" value="0.0" />
         <xacro:property name="imu_r" value="-3.1415" />
         <xacro:property name="imu_p" value="0.0" />
-        <xacro:property name="imu_y" value="-1.5708" />
+        <xacro:property name="imu_y" value="1.5708" />
       </xacro:unless>
     </xacro:if>
@@ -69,5 +69,5 @@
         <link name="${camera_name}_imu_frame" />
         <joint name="${camera_name}_imu_joint" type="fixed">
-            <parent link="${base_frame}"/>
+            <parent link="${camera_name}_right_camera_optical_frame"/>
             <child link="${camera_name}_imu_frame"/>
             <origin xyz="${imu_offset_x} ${imu_offset_y} ${imu_offset_z}" rpy="${imu_r} ${imu_p} ${imu_y}" />

Commit message: initial tf publisher

File: depthai_descriptions/urdf/include/depthai_macro.urdf.xacro (robot description, xacro)
@@ -53,43 +53,4 @@
         </joint>
     </xacro:if>
-<!-- RGB Camera -->
-    <link name="${camera_name}_rgb_camera_frame" />
-    <joint name="${camera_name}_rgb_camera_joint" type="fixed">
-        <parent link="${base_frame}"/>
-        <child link="${camera_name}_rgb_camera_frame"/>
-        <origin xyz="0 0 0" rpy="0 0 0" />
-    </joint>
-    <link name="${camera_name}_rgb_camera_optical_frame"/>
-    <joint name="${camera_name}_rgb_camera_optical_joint" type="fixed">
-        <origin xyz="0 0 0" rpy="-${M_PI/2} 0.0 -${M_PI/2}"/>
-        <parent link="${camera_name}_rgb_camera_frame"/>
-        <child link="${camera_name}_rgb_camera_optical_frame"/>
-    </joint>
-<!-- Left Camera -->
-    <link name="${camera_name}_left_camera_frame" />
-    <joint name="${camera_name}_left_camera_joint" type="fixed">
-        <parent link="${base_frame}"/>
-        <child link="${camera_name}_left_camera_frame"/>
-        <origin xyz="0 ${baseline/2} 0" rpy="0 0 0" />
-    </joint>
-    <link name="${camera_name}_left_camera_optical_frame"/>
-    <joint name="${camera_name}_left_camera_optical_joint" type="fixed">
-        <origin xyz="0 0 0" rpy="-${M_PI/2} 0.0 -${M_PI/2}"/>
-        <parent link="${camera_name}_left_camera_frame"/>
-        <child link="${camera_name}_left_camera_optical_frame"/>
-    </joint>
-<!-- right Camera -->
-    <link name="${camera_name}_right_camera_frame" />
-    <joint name="${camera_name}_right_camera_joint" type="fixed">
-        <parent link="${base_frame}"/>
-        <child link="${camera_name}_right_camera_frame"/>
-        <origin xyz="0 -${baseline/2} 0" rpy="0 0 0" />
-    </joint>
-    <link name="${camera_name}_right_camera_optical_frame"/>
-    <joint name="${camera_name}_right_camera_optical_joint" type="fixed">
-        <origin xyz="0 0 0" rpy="-${M_PI/2} 0.0 -${M_PI/2}"/>
-        <parent link="${camera_name}_right_camera_frame"/>
-        <child link="${camera_name}_right_camera_optical_frame"/>
-    </joint>
 </xacro:macro>
 </robot>

Commit message: add rsp via parameter setting

File: depthai_descriptions/urdf/include/depthai_macro.urdf.xacro (robot description, xacro)
@@ -53,4 +53,43 @@
         </joint>
     </xacro:if>
+<!-- RGB Camera -->
+    <link name="${camera_name}_rgb_camera_frame" />
+    <joint name="${camera_name}_rgb_camera_joint" type="fixed">
+        <parent link="${base_frame}"/>
+        <child link="${camera_name}_rgb_camera_frame"/>
+        <origin xyz="0 0 0" rpy="0 0 0" />
+    </joint>
+    <link name="${camera_name}_rgb_camera_optical_frame"/>
+    <joint name="${camera_name}_rgb_camera_optical_joint" type="fixed">
+        <origin xyz="0 0 0" rpy="-${M_PI/2} 0.0 -${M_PI/2}"/>
+        <parent link="${camera_name}_rgb_camera_frame"/>
+        <child link="${camera_name}_rgb_camera_optical_frame"/>
+    </joint>
+<!-- Left Camera -->
+    <link name="${camera_name}_left_camera_frame" />
+    <joint name="${camera_name}_left_camera_joint" type="fixed">
+        <parent link="${base_frame}"/>
+        <child link="${camera_name}_left_camera_frame"/>
+        <origin xyz="0 ${baseline/2} 0" rpy="0 0 0" />
+    </joint>
+    <link name="${camera_name}_left_camera_optical_frame"/>
+    <joint name="${camera_name}_left_camera_optical_joint" type="fixed">
+        <origin xyz="0 0 0" rpy="-${M_PI/2} 0.0 -${M_PI/2}"/>
+        <parent link="${camera_name}_left_camera_frame"/>
+        <child link="${camera_name}_left_camera_optical_frame"/>
+    </joint>
+<!-- right Camera -->
+    <link name="${camera_name}_right_camera_frame" />
+    <joint name="${camera_name}_right_camera_joint" type="fixed">
+        <parent link="${base_frame}"/>
+        <child link="${camera_name}_right_camera_frame"/>
+        <origin xyz="0 -${baseline/2} 0" rpy="0 0 0" />
+    </joint>
+    <link name="${camera_name}_right_camera_optical_frame"/>
+    <joint name="${camera_name}_right_camera_optical_joint" type="fixed">
+        <origin xyz="0 0 0" rpy="-${M_PI/2} 0.0 -${M_PI/2}"/>
+        <parent link="${camera_name}_right_camera_frame"/>
+        <child link="${camera_name}_right_camera_optical_frame"/>
+    </joint>
 </xacro:macro>
 </robot>

Commit message: added base urdf frame

File: depthai_descriptions/urdf/include/depthai_macro.urdf.xacro (robot description, xacro)
@@ -1,95 +1,26 @@
 <?xml version="1.0"?>
-<robot name="depthai_camera" xmlns:xacro="http://ros.org/wiki/xacro">
-<xacro:macro name="depthai_camera" params="camera_name camera_model parent base_frame
+<robot name="depthai_camera"
+    xmlns:xacro="http://ros.org/wiki/xacro">
+    <xacro:macro name="depthai_camera" params="camera_name camera_model parent base_frame
                                            cam_pos_x cam_pos_y cam_pos_z
-                                           cam_roll cam_pitch cam_yaw
-                                           r:=0.8 g:=0.8 b:=0.8 a:=0.8">
-    <xacro:property name="M_PI"     value="3.1415926535897931" />
-    <xacro:property name="model"    value="${camera_model}" />
-    <xacro:property name="has_imu" value="false" />
-    <!-- <xacro:if value="${model == 'BW1098OAK'}">
+                                           cam_roll cam_pitch cam_yaw r:=0.8 g:=0.8 b:=0.8 a:=0.8 ">
+        <xacro:include filename="$(find depthai_descriptions)/urdf/include/base_macro.urdf.xacro"/>
+        <xacro:property name="M_PI" value="3.1415926535897931" />
+        <xacro:property name="model" value="${camera_model}" />
+        <xacro:property name="has_imu" value="false" />
+        <!-- <xacro:if value="${model == 'BW1098OAK'}">
     </xacro:if> -->
-    <xacro:property name="baseline" value="0.075" />
-    <xacro:if value="${model == 'OAK-D'}">
-      <xacro:property name="has_imu" value="true" />
-      <xacro:property name="imu_offset_x" value="0.0" />
-      <xacro:property name="imu_offset_y" value="-0.015" />
-      <xacro:property name="imu_offset_z" value="-0.013662" />
-      <xacro:property name="imu_r" value="0" />
-      <xacro:property name="imu_p" value="1.5708" />
-      <xacro:property name="imu_y" value="0" />
-    </xacro:if>
-    <!-- base_link of the sensor-->
-    <link name="${base_frame}"/>
-    <joint name="${camera_name}_center_joint" type="fixed">
-        <parent link="${parent}"/>
-        <child link="${base_frame}"/>
-        <origin xyz="${cam_pos_x} ${cam_pos_y} ${cam_pos_z}" rpy="${cam_roll} ${cam_pitch} ${cam_yaw}" />
-    </joint>
-<!-- device Center -->
-    <link name="${camera_name}_model_origin">
-        <visual>
-            <origin xyz="0 0 0" rpy="0 0 0"/>
-            <geometry>
-                <mesh filename="package://depthai_descriptions/urdf/models/${model}.stl" />
-            </geometry>
-            <material name="mat">
-                <color rgba="${r} ${g} ${b} ${a}"/>
-            </material>
-        </visual>
-    </link>
-    <joint name="${camera_name}_model_origin_joint" type="fixed">
-        <parent link="${base_frame}"/>
-        <child link="${camera_name}_model_origin"/>
-        <origin xyz="0 0 0" rpy="1.5708 0 1.5708" />
-    </joint>
-<!-- IMU -->
-    <xacro:if value="${has_imu}">
-        <link name="${camera_name}_imu_frame" />
-        <joint name="${camera_name}_imu_joint" type="fixed">
-            <parent link="${base_frame}"/>
-            <child link="${camera_name}_imu_frame"/>
-            <origin xyz="${imu_offset_x} ${imu_offset_y} ${imu_offset_z}" rpy="${imu_r} ${imu_p} ${imu_y}" />
-        </joint>
-    </xacro:if>
-<!-- RGB Camera -->
-    <link name="${camera_name}_rgb_camera_frame" />
-    <joint name="${camera_name}_rgb_camera_joint" type="fixed">
-        <parent link="${base_frame}"/>
-        <child link="${camera_name}_rgb_camera_frame"/>
-        <origin xyz="0 0 0" rpy="0 0 0" />
-    </joint>
-    <link name="${camera_name}_rgb_camera_optical_frame"/>
-    <joint name="${camera_name}_rgb_camera_optical_joint" type="fixed">
-        <origin xyz="0 0 0" rpy="-${M_PI/2} 0.0 -${M_PI/2}"/>
-        <parent link="${camera_name}_rgb_camera_frame"/>
-        <child link="${camera_name}_rgb_camera_optical_frame"/>
-    </joint>
-<!-- Left Camera -->
-    <link name="${camera_name}_left_camera_frame" />
-    <joint name="${camera_name}_left_camera_joint" type="fixed">
-        <parent link="${base_frame}"/>
-        <child link="${camera_name}_left_camera_frame"/>
-        <origin xyz="0 ${baseline/2} 0" rpy="0 0 0" />
-    </joint>
-    <link name="${camera_name}_left_camera_optical_frame"/>
-    <joint name="${camera_name}_left_camera_optical_joint" type="fixed">
-        <origin xyz="0 0 0" rpy="-${M_PI/2} 0.0 -${M_PI/2}"/>
-        <parent link="${camera_name}_left_camera_frame"/>
-        <child link="${camera_name}_left_camera_optical_frame"/>
-    </joint>
-<!-- right Camera -->
-    <link name="${camera_name}_right_camera_frame" />
-    <joint name="${camera_name}_right_camera_joint" type="fixed">
-        <parent link="${base_frame}"/>
-        <child link="${camera_name}_right_camera_frame"/>
-        <origin xyz="0 -${baseline/2} 0" rpy="0 0 0" />
-    </joint>
-    <link name="${camera_name}_right_camera_optical_frame"/>
-    <joint name="${camera_name}_right_camera_optical_joint" type="fixed">
-        <origin xyz="0 0 0" rpy="-${M_PI/2} 0.0 -${M_PI/2}"/>
-        <parent link="${camera_name}_right_camera_frame"/>
-        <child link="${camera_name}_right_camera_optical_frame"/>
-    </joint>
-</xacro:macro>
+        <xacro:property name="baseline" value="0.075" />
+        <xacro:if value="${model == 'OAK-D'}">
+            <xacro:property name="has_imu" value="true" />
+            <xacro:property name="imu_offset_x" value="0.0" />
+            <xacro:property name="imu_offset_y" value="-0.015" />
+            <xacro:property name="imu_offset_z" value="-0.013662" />
+            <xacro:property name="imu_r" value="0" />
+            <xacro:property name="imu_p" value="1.5708" />
+            <xacro:property name="imu_y" value="0" />
+        </xacro:if>
+        <xacro:base camera_name = "$(arg camera_name)" parent = "$(arg parent_frame)" camera_model = "$(arg camera_model)" base_frame = "$(arg base_frame)" cam_pos_x = "$(arg cam_pos_x)" cam_pos_y = "$(arg cam_pos_y)" cam_pos_z = "$(arg cam_pos_z)" cam_roll = "$(arg cam_roll)" cam_pitch = "$(arg cam_pitch)" cam_yaw = "$(arg cam_yaw)"/>
+        <!-- IMU -->
+    </xacro:macro>
 </robot>

Commit message: return default sensor frames

File: depthai_descriptions/urdf/include/depthai_macro.urdf.xacro (robot description, xacro)
@@ -23,4 +23,51 @@
         <xacro:base camera_name = "$(arg camera_name)" parent = "$(arg parent_frame)" camera_model = "$(arg camera_model)" base_frame = "$(arg base_frame)" cam_pos_x = "$(arg cam_pos_x)" cam_pos_y = "$(arg cam_pos_y)" cam_pos_z = "$(arg cam_pos_z)" cam_roll = "$(arg cam_roll)" cam_pitch = "$(arg cam_pitch)" cam_yaw = "$(arg cam_yaw)"/>
         <!-- IMU -->
+        <xacro:if value="${has_imu}">
+            <link name="${camera_name}_imu_frame" />
+            <joint name="${camera_name}_imu_joint" type="fixed">
+                <parent link="${base_frame}"/>
+                <child link="${camera_name}_imu_frame"/>
+                <origin xyz="${imu_offset_x} ${imu_offset_y} ${imu_offset_z}" rpy="${imu_r} ${imu_p} ${imu_y}" />
+            </joint>
+        </xacro:if>
+        <!-- RGB Camera -->
+        <link name="${camera_name}_rgb_camera_frame" />
+        <joint name="${camera_name}_rgb_camera_joint" type="fixed">
+            <parent link="${base_frame}"/>
+            <child link="${camera_name}_rgb_camera_frame"/>
+            <origin xyz="0 0 0" rpy="0 0 0" />
+        </joint>
+        <link name="${camera_name}_rgb_camera_optical_frame"/>
+        <joint name="${camera_name}_rgb_camera_optical_joint" type="fixed">
+            <origin xyz="0 0 0" rpy="-${M_PI/2} 0.0 -${M_PI/2}"/>
+            <parent link="${camera_name}_rgb_camera_frame"/>
+            <child link="${camera_name}_rgb_camera_optical_frame"/>
+        </joint>
+        <!-- Left Camera -->
+        <link name="${camera_name}_left_camera_frame" />
+        <joint name="${camera_name}_left_camera_joint" type="fixed">
+            <parent link="${base_frame}"/>
+            <child link="${camera_name}_left_camera_frame"/>
+            <origin xyz="0 ${baseline/2} 0" rpy="0 0 0" />
+        </joint>
+        <link name="${camera_name}_left_camera_optical_frame"/>
+        <joint name="${camera_name}_left_camera_optical_joint" type="fixed">
+            <origin xyz="0 0 0" rpy="-${M_PI/2} 0.0 -${M_PI/2}"/>
+            <parent link="${camera_name}_left_camera_frame"/>
+            <child link="${camera_name}_left_camera_optical_frame"/>
+        </joint>
+        <!-- right Camera -->
+        <link name="${camera_name}_right_camera_frame" />
+        <joint name="${camera_name}_right_camera_joint" type="fixed">
+            <parent link="${base_frame}"/>
+            <child link="${camera_name}_right_camera_frame"/>
+            <origin xyz="0 -${baseline/2} 0" rpy="0 0 0" />
+        </joint>
+        <link name="${camera_name}_right_camera_optical_frame"/>
+        <joint name="${camera_name}_right_camera_optical_joint" type="fixed">
+            <origin xyz="0 0 0" rpy="-${M_PI/2} 0.0 -${M_PI/2}"/>
+            <parent link="${camera_name}_right_camera_frame"/>
+            <child link="${camera_name}_right_camera_optical_frame"/>
+        </joint>
     </xacro:macro>
 </robot>

Commit message: oak-d-sr-lr support

File: depthai_descriptions/urdf/include/depthai_macro.urdf.xacro (robot description, xacro)
@@ -10,4 +10,7 @@
         <xacro:property name="has_imu" value="false" />
         <xacro:property name="baseline" value="0.075" />
+        <xacro:if value="${model in ['OAK-D-SR']}">
+            <xacro:property name="baseline" value="0.02" />
+        </xacro:if>
         <xacro:if value="${model in ['OAK-D', 'OAK-D-PRO', 'OAK-D-POE']}">
             <xacro:property name="has_imu" value="true" />
@@ -15,16 +18,19 @@
         <xacro:base camera_name="${camera_name}" parent="${parent}" camera_model="${camera_model}" base_frame="${base_frame}" cam_pos_x="${cam_pos_x}" cam_pos_y="${cam_pos_y}" cam_pos_z="${cam_pos_z}" cam_roll="${cam_roll}" cam_pitch="${cam_pitch}" cam_yaw="${cam_yaw}" has_imu="${has_imu}"/>
         <!-- RGB Camera -->
-        <link name="${camera_name}_rgb_camera_frame" />
-        <joint name="${camera_name}_rgb_camera_joint" type="fixed">
-            <parent link="${base_frame}"/>
-            <child link="${camera_name}_rgb_camera_frame"/>
-            <origin xyz="0 0 0" rpy="0 0 0" />
-        </joint>
-        <link name="${camera_name}_rgb_camera_optical_frame"/>
-        <joint name="${camera_name}_rgb_camera_optical_joint" type="fixed">
-            <origin xyz="0 0 0" rpy="-${M_PI/2} 0.0 -${M_PI/2}"/>
-            <parent link="${camera_name}_rgb_camera_frame"/>
-            <child link="${camera_name}_rgb_camera_optical_frame"/>
-        </joint>
+        <xacro:unless value="${model in ['OAK-D-SR']}">
+            <link name="${camera_name}_rgb_camera_frame" />
+            <joint name="${camera_name}_rgb_camera_joint" type="fixed">
+                <parent link="${base_frame}"/>
+                <child link="${camera_name}_rgb_camera_frame"/>
+                <origin xyz="0 0 0" rpy="0 0 0" />
+            </joint>
+            <link name="${camera_name}_rgb_camera_optical_frame"/>
+            <joint name="${camera_name}_rgb_camera_optical_joint" type="fixed">
+                <origin xyz="0 0 0" rpy="-${M_PI/2} 0.0 -${M_PI/2}"/>
+                <parent link="${camera_name}_rgb_camera_frame"/>
+                <child link="${camera_name}_rgb_camera_optical_frame"/>
+            </joint>
+        </xacro:unless>
+        <xacro:unless value="${model in ['OAK-D-LR']}">
         <!-- Left Camera -->
         <link name="${camera_name}_left_camera_frame" />
@@ -53,4 +59,33 @@
             <child link="${camera_name}_right_camera_optical_frame"/>
         </joint>
+        </xacro:unless>
+        <xacro:if value="${model in ['OAK-D-LR']}">
+        <!-- left Camera -->
+        <link name="${camera_name}_left_camera_frame" />
+        <joint name="${camera_name}_left_camera_joint" type="fixed">
+            <parent link="${base_frame}"/>
+            <child link="${camera_name}_left_camera_frame"/>
+            <origin xyz="0 0.1 0" rpy="0 0 0" />
+        </joint>
+        <link name="${camera_name}_left_camera_optical_frame"/>
+        <joint name="${camera_name}_left_camera_optical_joint" type="fixed">
+            <origin xyz="0 0 0" rpy="-${M_PI/2} 0.0 -${M_PI/2}"/>
+            <parent link="${camera_name}_left_camera_frame"/>
+            <child link="${camera_name}_left_camera_optical_frame"/>
+        </joint>
+         <!-- right Camera -->
+        <link name="${camera_name}_right_camera_frame" />
+        <joint name="${camera_name}_right_camera_joint" type="fixed">
+            <parent link="${base_frame}"/>
+            <child link="${camera_name}_right_camera_frame"/>
+            <origin xyz="0 -0.05 0" rpy="0 0 0" />
+        </joint>
+        <link name="${camera_name}_right_camera_optical_frame"/>
+        <joint name="${camera_name}_right_camera_optical_joint" type="fixed">
+            <origin xyz="0 0 0" rpy="-${M_PI/2} 0.0 -${M_PI/2}"/>
+            <parent link="${camera_name}_right_camera_frame"/>
+            <child link="${camera_name}_right_camera_optical_frame"/>
+        </joint>
+    </xacro:if>
     </xacro:macro>
 </robot>

Commit message: fix urdf

File: depthai_descriptions/urdf/include/depthai_macro.urdf.xacro (robot description, xacro)
@@ -89,31 +89,3 @@
     </xacro:if>
     </xacro:macro>
-        <!-- right Camera -->
-        <link name="${camera_name}_right_camera_frame" />
-        <joint name="${camera_name}_right_camera_joint" type="fixed">
-            <parent link="${base_frame}"/>
-            <child link="${camera_name}_right_camera_frame"/>
-            <origin xyz="0 -${baseline/2} 0" rpy="0 0 0" />
-        </joint>
-        <link name="${camera_name}_right_camera_optical_frame"/>
-        <joint name="${camera_name}_right_camera_optical_joint" type="fixed">
-            <origin xyz="0 0 0" rpy="-${M_PI/2} 0.0 -${M_PI/2}"/>
-            <parent link="${camera_name}_right_camera_frame"/>
-            <child link="${camera_name}_right_camera_optical_frame"/>
-        </joint>
-    </xacro:macro>
-        <!-- right Camera -->
-        <link name="${camera_name}_right_camera_frame" />
-        <joint name="${camera_name}_right_camera_joint" type="fixed">
-            <parent link="${base_frame}"/>
-            <child link="${camera_name}_right_camera_frame"/>
-            <origin xyz="0 -${baseline/2} 0" rpy="0 0 0" />
-        </joint>
-        <link name="${camera_name}_right_camera_optical_frame"/>
-        <joint name="${camera_name}_right_camera_optical_joint" type="fixed">
-            <origin xyz="0 0 0" rpy="-${M_PI/2} 0.0 -${M_PI/2}"/>
-            <parent link="${camera_name}_right_camera_frame"/>
-            <child link="${camera_name}_right_camera_optical_frame"/>
-        </joint>
-    </xacro:macro>
 </robot>
