Commit message: SR-LR Update Iron (#482)

File: depthai_descriptions/urdf/include/depthai_macro.urdf.xacro (robot description, xacro)
@@ -10,4 +10,7 @@
         <xacro:property name="has_imu" value="false" />
         <xacro:property name="baseline" value="0.075" />
+        <xacro:if value="${model in ['OAK-D-SR']}">
+            <xacro:property name="baseline" value="0.02" />
+        </xacro:if>
         <xacro:if value="${model in ['OAK-D', 'OAK-D-PRO', 'OAK-D-POE']}">
             <xacro:property name="has_imu" value="true" />
@@ -15,16 +18,19 @@
         <xacro:base camera_name="${camera_name}" parent="${parent}" camera_model="${camera_model}" base_frame="${base_frame}" cam_pos_x="${cam_pos_x}" cam_pos_y="${cam_pos_y}" cam_pos_z="${cam_pos_z}" cam_roll="${cam_roll}" cam_pitch="${cam_pitch}" cam_yaw="${cam_yaw}" has_imu="${has_imu}"/>
         <!-- RGB Camera -->
-        <link name="${camera_name}_rgb_camera_frame" />
-        <joint name="${camera_name}_rgb_camera_joint" type="fixed">
-            <parent link="${base_frame}"/>
-            <child link="${camera_name}_rgb_camera_frame"/>
-            <origin xyz="0 0 0" rpy="0 0 0" />
-        </joint>
-        <link name="${camera_name}_rgb_camera_optical_frame"/>
-        <joint name="${camera_name}_rgb_camera_optical_joint" type="fixed">
-            <origin xyz="0 0 0" rpy="-${M_PI/2} 0.0 -${M_PI/2}"/>
-            <parent link="${camera_name}_rgb_camera_frame"/>
-            <child link="${camera_name}_rgb_camera_optical_frame"/>
-        </joint>
+        <xacro:unless value="${model in ['OAK-D-SR']}">
+            <link name="${camera_name}_rgb_camera_frame" />
+            <joint name="${camera_name}_rgb_camera_joint" type="fixed">
+                <parent link="${base_frame}"/>
+                <child link="${camera_name}_rgb_camera_frame"/>
+                <origin xyz="0 0 0" rpy="0 0 0" />
+            </joint>
+            <link name="${camera_name}_rgb_camera_optical_frame"/>
+            <joint name="${camera_name}_rgb_camera_optical_joint" type="fixed">
+                <origin xyz="0 0 0" rpy="-${M_PI/2} 0.0 -${M_PI/2}"/>
+                <parent link="${camera_name}_rgb_camera_frame"/>
+                <child link="${camera_name}_rgb_camera_optical_frame"/>
+            </joint>
+        </xacro:unless>
+        <xacro:unless value="${model in ['OAK-D-LR']}">
         <!-- Left Camera -->
         <link name="${camera_name}_left_camera_frame" />
@@ -53,11 +59,25 @@
             <child link="${camera_name}_right_camera_optical_frame"/>
         </joint>
-    </xacro:macro>
-        <!-- right Camera -->
+        </xacro:unless>
+        <xacro:if value="${model in ['OAK-D-LR']}">
+        <!-- left Camera -->
+        <link name="${camera_name}_left_camera_frame" />
+        <joint name="${camera_name}_left_camera_joint" type="fixed">
+            <parent link="${base_frame}"/>
+            <child link="${camera_name}_left_camera_frame"/>
+            <origin xyz="0 0.1 0" rpy="0 0 0" />
+        </joint>
+        <link name="${camera_name}_left_camera_optical_frame"/>
+        <joint name="${camera_name}_left_camera_optical_joint" type="fixed">
+            <origin xyz="0 0 0" rpy="-${M_PI/2} 0.0 -${M_PI/2}"/>
+            <parent link="${camera_name}_left_camera_frame"/>
+            <child link="${camera_name}_left_camera_optical_frame"/>
+        </joint>
+         <!-- right Camera -->
         <link name="${camera_name}_right_camera_frame" />
         <joint name="${camera_name}_right_camera_joint" type="fixed">
             <parent link="${base_frame}"/>
             <child link="${camera_name}_right_camera_frame"/>
-            <origin xyz="0 -${baseline/2} 0" rpy="0 0 0" />
+            <origin xyz="0 -0.05 0" rpy="0 0 0" />
         </joint>
         <link name="${camera_name}_right_camera_optical_frame"/>
@@ -67,4 +87,5 @@
             <child link="${camera_name}_right_camera_optical_frame"/>
         </joint>
+    </xacro:if>
     </xacro:macro>
 </robot>

Commit message: bump versions, update changelog & readme

File: depthai_descriptions/urdf/include/depthai_macro.urdf.xacro (robot description, xacro)
@@ -33,59 +33,59 @@
         </xacro:unless>
         <xacro:unless value="${model in ['OAK-D-LR']}">
-        <!-- Left Camera -->
-        <link name="${camera_name}_left_camera_frame" />
-        <joint name="${camera_name}_left_camera_joint" type="fixed">
-            <parent link="${base_frame}"/>
-            <child link="${camera_name}_left_camera_frame"/>
-            <origin xyz="0 ${baseline/2} 0" rpy="0 0 0" />
-        </joint>
-        <link name="${camera_name}_left_camera_optical_frame"/>
-        <joint name="${camera_name}_left_camera_optical_joint" type="fixed">
-            <origin xyz="0 0 0" rpy="-${M_PI/2} 0.0 -${M_PI/2}"/>
-            <parent link="${camera_name}_left_camera_frame"/>
-            <child link="${camera_name}_left_camera_optical_frame"/>
-        </joint>
-        <!-- right Camera -->
-        <link name="${camera_name}_right_camera_frame" />
-        <joint name="${camera_name}_right_camera_joint" type="fixed">
-            <parent link="${base_frame}"/>
-            <child link="${camera_name}_right_camera_frame"/>
-            <origin xyz="0 -${baseline/2} 0" rpy="0 0 0" />
-        </joint>
-        <link name="${camera_name}_right_camera_optical_frame"/>
-        <joint name="${camera_name}_right_camera_optical_joint" type="fixed">
-            <origin xyz="0 0 0" rpy="-${M_PI/2} 0.0 -${M_PI/2}"/>
-            <parent link="${camera_name}_right_camera_frame"/>
-            <child link="${camera_name}_right_camera_optical_frame"/>
-        </joint>
+            <!-- Left Camera -->
+            <link name="${camera_name}_left_camera_frame" />
+            <joint name="${camera_name}_left_camera_joint" type="fixed">
+                <parent link="${base_frame}"/>
+                <child link="${camera_name}_left_camera_frame"/>
+                <origin xyz="0 ${baseline/2} 0" rpy="0 0 0" />
+            </joint>
+            <link name="${camera_name}_left_camera_optical_frame"/>
+            <joint name="${camera_name}_left_camera_optical_joint" type="fixed">
+                <origin xyz="0 0 0" rpy="-${M_PI/2} 0.0 -${M_PI/2}"/>
+                <parent link="${camera_name}_left_camera_frame"/>
+                <child link="${camera_name}_left_camera_optical_frame"/>
+            </joint>
+            <!-- right Camera -->
+            <link name="${camera_name}_right_camera_frame" />
+            <joint name="${camera_name}_right_camera_joint" type="fixed">
+                <parent link="${base_frame}"/>
+                <child link="${camera_name}_right_camera_frame"/>
+                <origin xyz="0 -${baseline/2} 0" rpy="0 0 0" />
+            </joint>
+            <link name="${camera_name}_right_camera_optical_frame"/>
+            <joint name="${camera_name}_right_camera_optical_joint" type="fixed">
+                <origin xyz="0 0 0" rpy="-${M_PI/2} 0.0 -${M_PI/2}"/>
+                <parent link="${camera_name}_right_camera_frame"/>
+                <child link="${camera_name}_right_camera_optical_frame"/>
+            </joint>
         </xacro:unless>
         <xacro:if value="${model in ['OAK-D-LR']}">
-        <!-- left Camera -->
-        <link name="${camera_name}_left_camera_frame" />
-        <joint name="${camera_name}_left_camera_joint" type="fixed">
-            <parent link="${base_frame}"/>
-            <child link="${camera_name}_left_camera_frame"/>
-            <origin xyz="0 0.1 0" rpy="0 0 0" />
-        </joint>
-        <link name="${camera_name}_left_camera_optical_frame"/>
-        <joint name="${camera_name}_left_camera_optical_joint" type="fixed">
-            <origin xyz="0 0 0" rpy="-${M_PI/2} 0.0 -${M_PI/2}"/>
-            <parent link="${camera_name}_left_camera_frame"/>
-            <child link="${camera_name}_left_camera_optical_frame"/>
-        </joint>
-         <!-- right Camera -->
-        <link name="${camera_name}_right_camera_frame" />
-        <joint name="${camera_name}_right_camera_joint" type="fixed">
-            <parent link="${base_frame}"/>
-            <child link="${camera_name}_right_camera_frame"/>
-            <origin xyz="0 -0.05 0" rpy="0 0 0" />
-        </joint>
-        <link name="${camera_name}_right_camera_optical_frame"/>
-        <joint name="${camera_name}_right_camera_optical_joint" type="fixed">
-            <origin xyz="0 0 0" rpy="-${M_PI/2} 0.0 -${M_PI/2}"/>
-            <parent link="${camera_name}_right_camera_frame"/>
-            <child link="${camera_name}_right_camera_optical_frame"/>
-        </joint>
-    </xacro:if>
+            <!-- left Camera -->
+            <link name="${camera_name}_left_camera_frame" />
+            <joint name="${camera_name}_left_camera_joint" type="fixed">
+                <parent link="${base_frame}"/>
+                <child link="${camera_name}_left_camera_frame"/>
+                <origin xyz="0 0.1 0" rpy="0 0 0" />
+            </joint>
+            <link name="${camera_name}_left_camera_optical_frame"/>
+            <joint name="${camera_name}_left_camera_optical_joint" type="fixed">
+                <origin xyz="0 0 0" rpy="-${M_PI/2} 0.0 -${M_PI/2}"/>
+                <parent link="${camera_name}_left_camera_frame"/>
+                <child link="${camera_name}_left_camera_optical_frame"/>
+            </joint>
+            <!-- right Camera -->
+            <link name="${camera_name}_right_camera_frame" />
+            <joint name="${camera_name}_right_camera_joint" type="fixed">
+                <parent link="${base_frame}"/>
+                <child link="${camera_name}_right_camera_frame"/>
+                <origin xyz="0 -0.05 0" rpy="0 0 0" />
+            </joint>
+            <link name="${camera_name}_right_camera_optical_frame"/>
+            <joint name="${camera_name}_right_camera_optical_joint" type="fixed">
+                <origin xyz="0 0 0" rpy="-${M_PI/2} 0.0 -${M_PI/2}"/>
+                <parent link="${camera_name}_right_camera_frame"/>
+                <child link="${camera_name}_right_camera_optical_frame"/>
+            </joint>
+        </xacro:if>
     </xacro:macro>
 </robot>

Commit message: update urdf publishing with rs frame names

File: depthai_descriptions/urdf/include/depthai_macro.urdf.xacro (robot description, xacro)
@@ -1,91 +1,109 @@
 <?xml version="1.0"?>
 <robot name="depthai_camera"
-    xmlns:xacro="http://ros.org/wiki/xacro">
-    <xacro:macro name="depthai_camera" params="camera_name camera_model parent base_frame
+	xmlns:xacro="http://ros.org/wiki/xacro">
+	<xacro:macro name="depthai_camera"
+		params="camera_name camera_model parent base_frame
                                            cam_pos_x cam_pos_y cam_pos_z
-                                           cam_roll cam_pitch cam_yaw r:=0.8 g:=0.8 b:=0.8 a:=0.8 simulation:=false">
-        <xacro:include filename="$(find depthai_descriptions)/urdf/include/base_macro.urdf.xacro"/>
-        <xacro:property name="M_PI" value="3.1415926535897931" />
-        <xacro:property name="model" value="${camera_model}" />
-        <xacro:property name="has_imu" value="false" />
-        <xacro:property name="baseline" value="0.075" />
-        <xacro:if value="${model in ['OAK-D-SR']}">
-            <xacro:property name="baseline" value="0.02" />
-        </xacro:if>
-        <xacro:if value="${model in ['OAK-D', 'OAK-D-PRO', 'OAK-D-POE']}">
-            <xacro:property name="has_imu" value="true" />
-        </xacro:if>
-        <xacro:base camera_name="${camera_name}" parent="${parent}" camera_model="${camera_model}" base_frame="${base_frame}" cam_pos_x="${cam_pos_x}" cam_pos_y="${cam_pos_y}" cam_pos_z="${cam_pos_z}" cam_roll="${cam_roll}" cam_pitch="${cam_pitch}" cam_yaw="${cam_yaw}" has_imu="${has_imu}" simulation="${simulation}"/>
-        <!-- RGB Camera -->
-        <xacro:unless value="${model in ['OAK-D-SR']}">
-            <link name="${camera_name}_rgb_camera_frame" />
-            <joint name="${camera_name}_rgb_camera_joint" type="fixed">
-                <parent link="${base_frame}"/>
-                <child link="${camera_name}_rgb_camera_frame"/>
-                <origin xyz="0 0 0" rpy="0 0 0" />
-            </joint>
-            <link name="${camera_name}_rgb_camera_optical_frame"/>
-            <joint name="${camera_name}_rgb_camera_optical_joint" type="fixed">
-                <origin xyz="0 0 0" rpy="-${M_PI/2} 0.0 -${M_PI/2}"/>
-                <parent link="${camera_name}_rgb_camera_frame"/>
-                <child link="${camera_name}_rgb_camera_optical_frame"/>
-            </joint>
-        </xacro:unless>
-        <xacro:unless value="${model in ['OAK-D-LR']}">
-            <!-- Left Camera -->
-            <link name="${camera_name}_left_camera_frame" />
-            <joint name="${camera_name}_left_camera_joint" type="fixed">
-                <parent link="${base_frame}"/>
-                <child link="${camera_name}_left_camera_frame"/>
-                <origin xyz="0 ${baseline/2} 0" rpy="0 0 0" />
-            </joint>
-            <link name="${camera_name}_left_camera_optical_frame"/>
-            <joint name="${camera_name}_left_camera_optical_joint" type="fixed">
-                <origin xyz="0 0 0" rpy="-${M_PI/2} 0.0 -${M_PI/2}"/>
-                <parent link="${camera_name}_left_camera_frame"/>
-                <child link="${camera_name}_left_camera_optical_frame"/>
-            </joint>
-            <!-- right Camera -->
-            <link name="${camera_name}_right_camera_frame" />
-            <joint name="${camera_name}_right_camera_joint" type="fixed">
-                <parent link="${base_frame}"/>
-                <child link="${camera_name}_right_camera_frame"/>
-                <origin xyz="0 -${baseline/2} 0" rpy="0 0 0" />
-            </joint>
-            <link name="${camera_name}_right_camera_optical_frame"/>
-            <joint name="${camera_name}_right_camera_optical_joint" type="fixed">
-                <origin xyz="0 0 0" rpy="-${M_PI/2} 0.0 -${M_PI/2}"/>
-                <parent link="${camera_name}_right_camera_frame"/>
-                <child link="${camera_name}_right_camera_optical_frame"/>
-            </joint>
-        </xacro:unless>
-        <xacro:if value="${model in ['OAK-D-LR']}">
-            <!-- left Camera -->
-            <link name="${camera_name}_left_camera_frame" />
-            <joint name="${camera_name}_left_camera_joint" type="fixed">
-                <parent link="${base_frame}"/>
-                <child link="${camera_name}_left_camera_frame"/>
-                <origin xyz="0 0.1 0" rpy="0 0 0" />
-            </joint>
-            <link name="${camera_name}_left_camera_optical_frame"/>
-            <joint name="${camera_name}_left_camera_optical_joint" type="fixed">
-                <origin xyz="0 0 0" rpy="-${M_PI/2} 0.0 -${M_PI/2}"/>
-                <parent link="${camera_name}_left_camera_frame"/>
-                <child link="${camera_name}_left_camera_optical_frame"/>
-            </joint>
-            <!-- right Camera -->
-            <link name="${camera_name}_right_camera_frame" />
-            <joint name="${camera_name}_right_camera_joint" type="fixed">
-                <parent link="${base_frame}"/>
-                <child link="${camera_name}_right_camera_frame"/>
-                <origin xyz="0 -0.05 0" rpy="0 0 0" />
-            </joint>
-            <link name="${camera_name}_right_camera_optical_frame"/>
-            <joint name="${camera_name}_right_camera_optical_joint" type="fixed">
-                <origin xyz="0 0 0" rpy="-${M_PI/2} 0.0 -${M_PI/2}"/>
-                <parent link="${camera_name}_right_camera_frame"/>
-                <child link="${camera_name}_right_camera_optical_frame"/>
-            </joint>
-        </xacro:if>
-    </xacro:macro>
+                                           cam_roll cam_pitch cam_yaw r:=0.8 g:=0.8 b:=0.8 a:=0.8 simulation:=false rs_compat:=false">
+		<xacro:include filename="$(find depthai_descriptions)/urdf/include/base_macro.urdf.xacro" />
+		<xacro:property name="M_PI" value="3.1415926535897931" />
+		<xacro:property name="model" value="${camera_model}" />
+		<xacro:property name="has_imu" value="false" />
+		<xacro:property name="baseline" value="0.075" />
+		<xacro:if value="${rs_compat}">
+			<xacro:property name="frame_suffix" value="frame" />
+			<xacro:property name="optical_frame_suffix" value="optical_frame" />
+			<xacro:property name="rgb_name" value="color" />
+			<xacro:property name="left_name" value="infra2" />
+			<xacro:property name="right_name" value="infra1" />
+		</xacro:if>
+		<xacro:unless value="${rs_compat}">
+			<xacro:property name="frame_suffix" value="camera_frame" />
+			<xacro:property name="optical_frame_suffix" value="camera_optical_frame" />
+			<xacro:property name="rgb_name" value="rgb" />
+			<xacro:property name="left_name" value="left" />
+			<xacro:property name="right_name" value="right" />
+		</xacro:unless>
+		<xacro:if value="${model in ['OAK-D-SR']}">
+			<xacro:property name="baseline" value="0.02" />
+		</xacro:if>
+		<xacro:if value="${model in ['OAK-D', 'OAK-D-PRO', 'OAK-D-POE']}">
+			<xacro:property name="has_imu" value="true" />
+		</xacro:if>
+		<xacro:base camera_name="${camera_name}" parent="${parent}" camera_model="${camera_model}"
+			base_frame="${base_frame}" cam_pos_x="${cam_pos_x}" cam_pos_y="${cam_pos_y}"
+			cam_pos_z="${cam_pos_z}" cam_roll="${cam_roll}" cam_pitch="${cam_pitch}"
+			cam_yaw="${cam_yaw}" has_imu="${has_imu}" simulation="${simulation}" />
+		<!-- RGB Camera -->
+		<xacro:unless value="${model in ['OAK-D-SR']}">
+			<link name="${camera_name}_${rgb_name}_${frame_suffix}" />
+			<joint name="${camera_name}_rgb_camera_joint" type="fixed">
+				<parent link="${base_frame}" />
+				<child link="${camera_name}_${rgb_name}_${frame_suffix}" />
+				<origin xyz="0 0 0" rpy="0 0 0" />
+			</joint>
+			<link name="${camera_name}_${rgb_name}_${optical_frame_suffix}" />
+			<joint name="${camera_name}_rgb_camera_optical_joint" type="fixed">
+				<origin xyz="0 0 0" rpy="-${M_PI/2} 0.0 -${M_PI/2}" />
+				<parent link="${camera_name}_${rgb_name}_${frame_suffix}" />
+				<child link="${camera_name}_${rgb_name}_${optical_frame_suffix}" />
+			</joint>
+		</xacro:unless>
+		<xacro:unless value="${model in ['OAK-D-LR']}">
+			<!-- Left Camera -->
+			<link name="${camera_name}_${left_name}_${frame_suffix}" />
+			<joint name="${camera_name}_left_camera_joint" type="fixed">
+				<parent link="${base_frame}" />
+				<child link="${camera_name}_${left_name}_${frame_suffix}" />
+				<origin xyz="0 ${baseline/2} 0" rpy="0 0 0" />
+			</joint>
+			<link name="${camera_name}_${left_name}_${optical_frame_suffix}" />
+			<joint name="${camera_name}_left_camera_optical_joint" type="fixed">
+				<origin xyz="0 0 0" rpy="-${M_PI/2} 0.0 -${M_PI/2}" />
+				<parent link="${camera_name}_${left_name}_${frame_suffix}" />
+				<child link="${camera_name}_${left_name}_${optical_frame_suffix}" />
+			</joint>
+			<!-- right Camera -->
+			<link name="${camera_name}_${right_name}_${frame_suffix}" />
+			<joint name="${camera_name}_right_camera_joint" type="fixed">
+				<parent link="${base_frame}" />
+				<child link="${camera_name}_${right_name}_${frame_suffix}" />
+				<origin xyz="0 -${baseline/2} 0" rpy="0 0 0" />
+			</joint>
+			<link name="${camera_name}_${right_name}_${optical_frame_suffix}" />
+			<joint name="${camera_name}_right_camera_optical_joint" type="fixed">
+				<origin xyz="0 0 0" rpy="-${M_PI/2} 0.0 -${M_PI/2}" />
+				<parent link="${camera_name}_${right_name}_${frame_suffix}" />
+				<child link="${camera_name}_${right_name}_${optical_frame_suffix}" />
+			</joint>
+		</xacro:unless>
+		<xacro:if value="${model in ['OAK-D-LR']}">
+			<!-- left Camera -->
+			<link name="${camera_name}_${left_name}_${frame_suffix}" />
+			<joint name="${camera_name}_left_camera_joint" type="fixed">
+				<parent link="${base_frame}" />
+				<child link="${camera_name}_${left_name}_${frame_suffix}" />
+				<origin xyz="0 0.1 0" rpy="0 0 0" />
+			</joint>
+			<link name="${camera_name}_${left_name}_${optical_frame_suffix}" />
+			<joint name="${camera_name}_left_camera_optical_joint" type="fixed">
+				<origin xyz="0 0 0" rpy="-${M_PI/2} 0.0 -${M_PI/2}" />
+				<parent link="${camera_name}_${left_name}_${frame_suffix}" />
+				<child link="${camera_name}_${left_name}_${optical_frame_suffix}" />
+			</joint>
+			<!-- right Camera -->
+			<link name="${camera_name}_${right_name}_${frame_suffix}" />
+			<joint name="${camera_name}_right_camera_joint" type="fixed">
+				<parent link="${base_frame}" />
+				<child link="${camera_name}_${right_name}_${frame_suffix}" />
+				<origin xyz="0 -0.05 0" rpy="0 0 0" />
+			</joint>
+			<link name="${camera_name}_${right_name}_${optical_frame_suffix}" />
+			<joint name="${camera_name}_right_camera_optical_joint" type="fixed">
+				<origin xyz="0 0 0" rpy="-${M_PI/2} 0.0 -${M_PI/2}" />
+				<parent link="${camera_name}_${right_name}_${frame_suffix}" />
+				<child link="${camera_name}_${right_name}_${optical_frame_suffix}" />
+			</joint>
+		</xacro:if>
+	</xacro:macro>
 </robot>

Commit message: updates after merge

File: depthai_descriptions/urdf/include/depthai_macro.urdf.xacro (robot description, xacro)
@@ -136,10 +136,3 @@
 		</xacro:if>
 	</xacro:macro>
-            <link name="${camera_name}_right_camera_optical_frame"/>
-            <joint name="${camera_name}_right_camera_optical_joint" type="fixed">
-                <origin xyz="0 0 0" rpy="-${M_PI/2} 0.0 -${M_PI/2}"/>
-                <parent link="${camera_name}_right_camera_frame"/>
-                <child link="${camera_name}_right_camera_optical_frame"/>
-            </joint>
-        </xacro:if>
-    </xacro:macro>
+</robot>
