Commit message: Fix description compatibility and driver save/shutdown crashes

File: depthai_descriptions/urdf/include/depthai_macro.urdf.xacro (robot description, xacro)
@@ -40,11 +40,11 @@
     </xacro:macro>
     <!-- Recursive expansion preserves extra sockets on boards with >3 cameras. -->
-	<xacro:macro name="depthai_extra_cameras" params="names cameras camera_name base_frame frame_suffix optical_frame_suffix socket_names aliases">
+	<xacro:macro name="depthai_extra_cameras" params="names cameras camera_name base_frame frame_suffix optical_frame_suffix socket_names aliases reserved_names">
 		<xacro:if value="${len(names) > 0}">
 			<xacro:property name="sensor" value="${names[0]}" />
 			<xacro:depthai_camera_frame camera_name="${camera_name}" base_frame="${base_frame}"
 				sensor_name="${socket_names.get(cameras[sensor]['socket'], sensor)}" joint_name="${sensor}" xyz="${cameras[sensor]['xyz']}"
-				rpy="${cameras[sensor]['rpy']}" aliases="${aliases}" legacy_name="${sensor}" reserved_names="${list(socket_names.values())}" frame_suffix="${frame_suffix}" optical_frame_suffix="${optical_frame_suffix}" />
-			<xacro:depthai_extra_cameras names="${names[1:]}" aliases="${aliases}" cameras="${cameras}" socket_names="${socket_names}" camera_name="${camera_name}"
+				rpy="${cameras[sensor]['rpy']}" aliases="${aliases}" legacy_name="${sensor}" reserved_names="${reserved_names}" frame_suffix="${frame_suffix}" optical_frame_suffix="${optical_frame_suffix}" />
+			<xacro:depthai_extra_cameras names="${names[1:]}" aliases="${aliases}" reserved_names="${reserved_names}" cameras="${cameras}" socket_names="${socket_names}" camera_name="${camera_name}"
 				base_frame="${base_frame}" frame_suffix="${frame_suffix}" optical_frame_suffix="${optical_frame_suffix}" />
 		</xacro:if>
@@ -78,4 +78,8 @@
 			<xacro:property name="socket_names" value="${dict(CAM_A='rgb', CAM_B='left', CAM_C='right', CAM_D='left_back', CAM_E='thermal')}" />
 		</xacro:if>
+        <!-- Only actual sockets can occupy an alias; absent standard sockets
+             must not suppress role aliases on sparse/nonstandard boards. -->
+        <xacro:property name="active_sockets" value="${[device_config.get(role + '_socket') for role in ['rgb', 'left', 'right'] if device_config.get(role + '_socket')] + [pose['socket'] for pose in device_config['extra_cameras'].values()]}" />
+        <xacro:property name="reserved_names" value="${[socket_names.get(socket, socket.lower()) for socket in active_sockets]}" />
 		<xacro:base camera_name="${camera_name}" parent="${parent}" camera_model="${camera_model}"
 			base_frame="${base_frame}" cam_pos_x="${cam_pos_x}" cam_pos_y="${cam_pos_y}"
@@ -84,19 +88,19 @@
 		<xacro:if value="${device_config['rgb_xyz'] is not None}">
 			<xacro:depthai_camera_frame camera_name="${camera_name}" base_frame="${base_frame}"
-				sensor_name="${socket_names.get(device_config.get('rgb_socket'), rgb_name)}" joint_name="rgb" aliases="${legacy_frame_aliases and not device_config['legacy']}" legacy_name="${rgb_name}" reserved_names="${list(socket_names.values())}" xyz="${device_config['rgb_xyz']}" rpy="${device_config['rgb_rpy']}"
+				sensor_name="${socket_names.get(device_config.get('rgb_socket'), rgb_name)}" joint_name="rgb" aliases="${legacy_frame_aliases and not device_config['legacy']}" legacy_name="${rgb_name}" reserved_names="${reserved_names}" xyz="${device_config['rgb_xyz']}" rpy="${device_config['rgb_rpy']}"
 				frame_suffix="${frame_suffix}" optical_frame_suffix="${optical_frame_suffix}" />
 		</xacro:if>
 		<xacro:if value="${device_config['left_xyz'] is not None}">
 			<xacro:depthai_camera_frame camera_name="${camera_name}" base_frame="${base_frame}"
-				sensor_name="${socket_names.get(device_config.get('left_socket'), left_name)}" joint_name="left" aliases="${legacy_frame_aliases and not device_config['legacy']}" legacy_name="${left_name}" reserved_names="${list(socket_names.values())}" xyz="${device_config['left_xyz']}" rpy="${device_config['left_rpy']}"
+				sensor_name="${socket_names.get(device_config.get('left_socket'), left_name)}" joint_name="left" aliases="${legacy_frame_aliases and not device_config['legacy']}" legacy_name="${left_name}" reserved_names="${reserved_names}" xyz="${device_config['left_xyz']}" rpy="${device_config['left_rpy']}"
 				frame_suffix="${frame_suffix}" optical_frame_suffix="${optical_frame_suffix}" />
 		</xacro:if>
 		<xacro:if value="${device_config['right_xyz'] is not None}">
 			<xacro:depthai_camera_frame camera_name="${camera_name}" base_frame="${base_frame}"
-				sensor_name="${device_config['right_name'] or socket_names.get(device_config.get('right_socket'), right_name)}" joint_name="right" aliases="${legacy_frame_aliases and not device_config['legacy']}" legacy_name="${'cam_e' if camera_model == 'OAK-T' else right_name}" reserved_names="${list(socket_names.values())}" xyz="${device_config['right_xyz']}" rpy="${device_config['right_rpy']}"
+				sensor_name="${device_config['right_name'] or socket_names.get(device_config.get('right_socket'), right_name)}" joint_name="right" aliases="${legacy_frame_aliases and not device_config['legacy']}" legacy_name="${'cam_e' if camera_model == 'OAK-T' else right_name}" reserved_names="${reserved_names}" xyz="${device_config['right_xyz']}" rpy="${device_config['right_rpy']}"
 				frame_suffix="${frame_suffix}" optical_frame_suffix="${optical_frame_suffix}" />
 		</xacro:if>
 		<xacro:depthai_extra_cameras names="${list(device_config['extra_cameras'].keys())}"
-			cameras="${device_config['extra_cameras']}" aliases="${legacy_frame_aliases and not device_config['legacy']}" socket_names="${socket_names}" camera_name="${camera_name}" base_frame="${base_frame}"
+			cameras="${device_config['extra_cameras']}" reserved_names="${reserved_names}" aliases="${legacy_frame_aliases and not device_config['legacy']}" socket_names="${socket_names}" camera_name="${camera_name}" base_frame="${base_frame}"
 			frame_suffix="${frame_suffix}" optical_frame_suffix="${optical_frame_suffix}" />
 	</xacro:macro>
