Commit message: additional IMU poses

File: depthai_descriptions/urdf/include/base_macro.urdf.xacro (robot description, xacro)
@@ -40,4 +40,20 @@
             <xacro:property name="imu_y" value="0" />
         </xacro:if>
+        <xacro:if value="${model == 'OAK-D-PRO'}">
+            <xacro:property name="imu_offset_x" value="-0.008" />
+            <xacro:property name="imu_offset_y" value="-0.037945" />
+            <xacro:property name="imu_offset_z" value="-0.00079" />
+            <xacro:property name="imu_r" value="{M_PI}" />
+            <xacro:property name="imu_p" value="${M_PI/2}" />
+            <xacro:property name="imu_y" value="0" />
+        </xacro:if>
+        <xacro:if value"${model == 'OAK-D-POE'}">
+            <xacro:property name="imu_offset_x" value="-0.008" />
+            <xacro:property name="imu_offset_y" value="-0.04" />
+            <xacro:property name="imu_offset_z" value="-0.020265" />
+            <xacro:property name="imu_r" value="{M_PI}" />
+            <xacro:property name="imu_p" value="${M_PI/2}" />
+            <xacro:property name="imu_y" value="0" />
+        </xacro:if>
         <xacro:if value="${has_imu}">
             <link name="${camera_name}_imu_frame" />

Commit message: fixed urdf

File: depthai_descriptions/urdf/include/base_macro.urdf.xacro (robot description, xacro)
@@ -36,7 +36,7 @@
             <xacro:property name="imu_offset_y" value="-0.015" />
             <xacro:property name="imu_offset_z" value="-0.013662" />
-            <xacro:property name="imu_r" value="0" />
-            <xacro:property name="imu_p" value="1.5708" />
-            <xacro:property name="imu_y" value="0" />
+            <xacro:property name="imu_r" value="0.0" />
+            <xacro:property name="imu_p" value="${M_PI/2.0}" />
+            <xacro:property name="imu_y" value="0.0" />
         </xacro:if>
         <xacro:if value="${model == 'OAK-D-PRO'}">
@@ -44,15 +44,15 @@
             <xacro:property name="imu_offset_y" value="-0.037945" />
             <xacro:property name="imu_offset_z" value="-0.00079" />
-            <xacro:property name="imu_r" value="{M_PI}" />
-            <xacro:property name="imu_p" value="${M_PI/2}" />
-            <xacro:property name="imu_y" value="0" />
+            <xacro:property name="imu_r" value="${M_PI}" />
+            <xacro:property name="imu_p" value="${M_PI/2.0}" />
+            <xacro:property name="imu_y" value="0.0" />
         </xacro:if>
-        <xacro:if value"${model == 'OAK-D-POE'}">
+        <xacro:if value="${model == 'OAK-D-POE'}">
             <xacro:property name="imu_offset_x" value="-0.008" />
             <xacro:property name="imu_offset_y" value="-0.04" />
             <xacro:property name="imu_offset_z" value="-0.020265" />
-            <xacro:property name="imu_r" value="{M_PI}" />
-            <xacro:property name="imu_p" value="${M_PI/2}" />
-            <xacro:property name="imu_y" value="0" />
+            <xacro:property name="imu_r" value="${M_PI}" />
+            <xacro:property name="imu_p" value="${M_PI/2.0}" />
+            <xacro:property name="imu_y" value="0.0" />
         </xacro:if>
         <xacro:if value="${has_imu}">

Commit message: Add Sr and Lr (BNO) imu to urdf

File: depthai_descriptions/urdf/include/base_macro.urdf.xacro (robot description, xacro)
@@ -56,4 +56,20 @@
             <xacro:property name="imu_y" value="0.0" />
         </xacro:if>
+        <xacro:if value="${model == 'OAK-D-LR'}">
+            <xacro:property name="imu_offset_x" value="0.0" />
+            <xacro:property name="imu_offset_y" value="-0.021443" />
+            <xacro:property name="imu_offset_z" value="-0.012614" />
+            <xacro:property name="imu_r" value="-${M_PI/2.0}" />
+            <xacro:property name="imu_p" value="0.0" />
+            <xacro:property name="imu_y" value="-${M_PI/2.0}" />
+        </xacro:if>
+        <xacro:if value="${model == 'OAK-D-SR'}">
+            <xacro:property name="imu_offset_x" value="0.0" />
+            <xacro:property name="imu_offset_y" value="0.00175" />
+            <xacro:property name="imu_offset_z" value="0.01713" />
+            <xacro:property name="imu_r" value="${M_PI/2.0}" />
+            <xacro:property name="imu_p" value="0.0" />
+            <xacro:property name="imu_y" value="${M_PI/2.0}" />
+        </xacro:if>
         <xacro:if value="${has_imu}">
             <link name="${camera_name}_imu_frame" />

File: depthai_descriptions/urdf/include/depthai_macro.urdf.xacro (robot description, xacro)
@@ -13,5 +13,5 @@
             <xacro:property name="baseline" value="0.02" />
         </xacro:if>
-        <xacro:if value="${model in ['OAK-D', 'OAK-D-PRO', 'OAK-D-POE']}">
+        <xacro:if value="${model in ['OAK-D', 'OAK-D-PRO', 'OAK-D-POE', 'OAK-D-SR', 'OAK-D-LR']}">
             <xacro:property name="has_imu" value="true" />
         </xacro:if>

Commit message: Use packages to find mesh at run time

File: depthai_descriptions/urdf/include/base_macro.urdf.xacro (robot description, xacro)
@@ -19,5 +19,5 @@
                 <origin xyz="0 0 0" rpy="0 0 0"/>
                 <geometry>
-                    <mesh filename="file://$(find depthai_descriptions)/urdf/models/${model}.stl" />
+                    <mesh filename="package://depthai_descriptions/urdf/models/${model}.stl" />
                 </geometry>
                 <material name="mat">

Commit message: add stl, update urdf and tof nodes for new api

File: depthai_descriptions/urdf/include/base_macro.urdf.xacro (robot description, xacro)
@@ -1,79 +1,97 @@
 <?xml version="1.0"?>
 <robot name="base"
-    xmlns:xacro="http://ros.org/wiki/xacro">
-    <xacro:macro name="base" params="camera_name camera_model parent base_frame
+	xmlns:xacro="http://ros.org/wiki/xacro">
+	<xacro:macro name="base"
+		params="camera_name camera_model parent base_frame
                                            cam_pos_x cam_pos_y cam_pos_z
                                            cam_roll cam_pitch cam_yaw has_imu r:=0.8 g:=0.8 b:=0.8 a:=0.8 simulation:=false">
-        <xacro:if value="${simulation}">
-            <xacro:property
-            name="file_prefix"
-            value="file://$(find depthai_descriptions)"
-            />
-        </xacro:if>
-        <xacro:unless value="${simulation}">
-            <xacro:property
-            name="file_prefix"
-            value="package://depthai_descriptions"
-            />
-        </xacro:unless>
-        <!-- base_link of the sensor-->
-        <link name="${base_frame}"/>
-        <xacro:property name="M_PI" value="3.1415926535897931" />
-        <xacro:property name="model" value="${camera_model}" />
-        <joint name="${camera_name}_center_joint" type="fixed">
-            <parent link="${parent}"/>
-            <child link="${base_frame}"/>
-            <origin xyz="${cam_pos_x} ${cam_pos_y} ${cam_pos_z}" rpy="${cam_roll} ${cam_pitch} ${cam_yaw}" />
-        </joint>
-        <!-- device Center -->
-        <link name="${camera_name}_model_origin">
-            <visual>
-                <origin xyz="0 0 0" rpy="0 0 0"/>
-                <geometry>
-                    <mesh filename="${file_prefix}/urdf/models/${model}.stl" />
-                </geometry>
-                <material name="mat">
-                    <color rgba="${r} ${g} ${b} ${a}"/>
-                </material>
-            </visual>
-        </link>
-        <joint name="${camera_name}_model_origin_joint" type="fixed">
-            <parent link="${base_frame}"/>
-            <child link="${camera_name}_model_origin"/>
-            <origin xyz="0 0 0" rpy="1.5708 0 1.5708" />
-        </joint>
-        <!-- IMU -->
-        <xacro:if value="${model == 'OAK-D'}">
-            <xacro:property name="imu_offset_x" value="0.0" />
-            <xacro:property name="imu_offset_y" value="-0.015" />
-            <xacro:property name="imu_offset_z" value="-0.013662" />
-            <xacro:property name="imu_r" value="0.0" />
-            <xacro:property name="imu_p" value="${M_PI/2.0}" />
-            <xacro:property name="imu_y" value="0.0" />
-        </xacro:if>
-        <xacro:if value="${model == 'OAK-D-PRO'}">
-            <xacro:property name="imu_offset_x" value="-0.008" />
-            <xacro:property name="imu_offset_y" value="-0.037945" />
-            <xacro:property name="imu_offset_z" value="-0.00079" />
-            <xacro:property name="imu_r" value="${M_PI}" />
-            <xacro:property name="imu_p" value="${M_PI/2.0}" />
-            <xacro:property name="imu_y" value="0.0" />
-        </xacro:if>
-        <xacro:if value="${model == 'OAK-D-POE'}">
-            <xacro:property name="imu_offset_x" value="-0.008" />
-            <xacro:property name="imu_offset_y" value="-0.04" />
-            <xacro:property name="imu_offset_z" value="-0.020265" />
-            <xacro:property name="imu_r" value="${M_PI}" />
-            <xacro:property name="imu_p" value="${M_PI/2.0}" />
-            <xacro:property name="imu_y" value="0.0" />
-        </xacro:if>
-        <xacro:if value="${has_imu}">
-            <link name="${camera_name}_imu_frame" />
-            <joint name="${camera_name}_imu_joint" type="fixed">
-                <parent link="${base_frame}"/>
-                <child link="${camera_name}_imu_frame"/>
-                <origin xyz="${imu_offset_x} ${imu_offset_y} ${imu_offset_z}" rpy="${imu_r} ${imu_p} ${imu_y}" />
-            </joint>
-        </xacro:if>
-    </xacro:macro>
+		<xacro:if value="${simulation}">
+			<xacro:property
+				name="file_prefix"
+				value="file://$(find depthai_descriptions)"
+			/>
+		</xacro:if>
+		<xacro:unless value="${simulation}">
+			<xacro:property
+				name="file_prefix"
+				value="package://depthai_descriptions"
+			/>
+		</xacro:unless>
+		<!-- base_link of the sensor-->
+		<link name="${base_frame}" />
+		<xacro:property name="M_PI" value="3.1415926535897931" />
+		<xacro:property name="model" value="${camera_model}" />
+		<joint name="${camera_name}_center_joint" type="fixed">
+			<parent link="${parent}" />
+			<child link="${base_frame}" />
+			<origin xyz="${cam_pos_x} ${cam_pos_y} ${cam_pos_z}"
+				rpy="${cam_roll} ${cam_pitch} ${cam_yaw}" />
+		</joint>
+		<!-- device Center -->
+		<xacro:unless value="${model in ['OAK-D-SR-POE']}">
+			<link name="${camera_name}_model_origin">
+				<visual>
+					<origin xyz="0 0 0" rpy="0 0 0" />
+					<geometry>
+						<mesh filename="${file_prefix}/urdf/models/${model}.stl" />
+					</geometry>
+					<material name="mat">
+						<color rgba="${r} ${g} ${b} ${a}" />
+					</material>
+				</visual>
+			</link>
+		</xacro:unless>
+		<xacro:if value="${model in ['OAK-D-SR-POE']}">
+			<link name="${camera_name}_model_origin">
+				<visual>
+					<origin xyz="0.019 0 0" rpy="0 0 0" />
+					<geometry>
+						<mesh filename="${file_prefix}/urdf/models/${model}.stl" />
+					</geometry>
+					<material name="mat">
+						<color rgba="${r} ${g} ${b} ${a}" />
+					</material>
+				</visual>
+			</link>
+		</xacro:if>
+		<joint name="${camera_name}_model_origin_joint" type="fixed">
+			<parent link="${base_frame}" />
+			<child link="${camera_name}_model_origin" />
+			<origin xyz="0 0 0" rpy="1.5708 0 1.5708" />
+		</joint>
+		<!-- IMU -->
+		<xacro:if value="${model == 'OAK-D'}">
+			<xacro:property name="imu_offset_x" value="0.0" />
+			<xacro:property name="imu_offset_y" value="-0.015" />
+			<xacro:property name="imu_offset_z" value="-0.013662" />
+			<xacro:property name="imu_r" value="0.0" />
+			<xacro:property name="imu_p" value="${M_PI/2.0}" />
+			<xacro:property name="imu_y" value="0.0" />
+		</xacro:if>
+		<xacro:if value="${model == 'OAK-D-PRO'}">
+			<xacro:property name="imu_offset_x" value="-0.008" />
+			<xacro:property name="imu_offset_y" value="-0.037945" />
+			<xacro:property name="imu_offset_z" value="-0.00079" />
+			<xacro:property name="imu_r" value="${M_PI}" />
+			<xacro:property name="imu_p" value="${M_PI/2.0}" />
+			<xacro:property name="imu_y" value="0.0" />
+		</xacro:if>
+		<xacro:if value="${model == 'OAK-D-POE'}">
+			<xacro:property name="imu_offset_x" value="-0.008" />
+			<xacro:property name="imu_offset_y" value="-0.04" />
+			<xacro:property name="imu_offset_z" value="-0.020265" />
+			<xacro:property name="imu_r" value="${M_PI}" />
+			<xacro:property name="imu_p" value="${M_PI/2.0}" />
+			<xacro:property name="imu_y" value="0.0" />
+		</xacro:if>
+		<xacro:if value="${has_imu}">
+			<link name="${camera_name}_imu_frame" />
+			<joint name="${camera_name}_imu_joint" type="fixed">
+				<parent link="${base_frame}" />
+				<child link="${camera_name}_imu_frame" />
+				<origin xyz="${imu_offset_x} ${imu_offset_y} ${imu_offset_z}"
+					rpy="${imu_r} ${imu_p} ${imu_y}" />
+			</joint>
+		</xacro:if>
+	</xacro:macro>
 </robot>

File: depthai_descriptions/urdf/include/depthai_macro.urdf.xacro (robot description, xacro)
@@ -50,5 +50,6 @@
 			</joint>
 		</xacro:unless>
-		<xacro:unless value="${model in ['OAK-D-LR']}">
+		<!-- LR and SR POE have different baselines and positions -->
+		<xacro:unless value="${model in ['OAK-D-LR', 'OAK-D-SR-POE']}">
 			<!-- Left Camera -->
 			<link name="${camera_name}_${left_name}_${frame_suffix}" />
@@ -106,4 +107,32 @@
 			</joint>
 		</xacro:if>
+		<xacro:if value="${model in ['OAK-D-SR-POE']}">
+			<!-- left Camera -->
+			<link name="${camera_name}_${left_name}_${frame_suffix}" />
+			<joint name="${camera_name}_left_camera_joint" type="fixed">
+				<parent link="${base_frame}" />
+				<child link="${camera_name}_${left_name}_${frame_suffix}" />
+				<origin xyz="0 0.0375 0" rpy="0 0 0" />
+			</joint>
+			<link name="${camera_name}_${left_name}_${optical_frame_suffix}" />
+			<joint name="${camera_name}_left_camera_optical_joint" type="fixed">
+				<origin xyz="0 0 0" rpy="-${M_PI/2} 0.0 -${M_PI/2}" />
+				<parent link="${camera_name}_${left_name}_${frame_suffix}" />
+				<child link="${camera_name}_${left_name}_${optical_frame_suffix}" />
+			</joint>
+			<!-- right Camera -->
+			<link name="${camera_name}_${right_name}_${frame_suffix}" />
+			<joint name="${camera_name}_right_camera_joint" type="fixed">
+				<parent link="${base_frame}" />
+				<child link="${camera_name}_${right_name}_${frame_suffix}" />
+				<origin xyz="0 0.0175 0" rpy="0 0 0" />
+			</joint>
+			<link name="${camera_name}_${right_name}_${optical_frame_suffix}" />
+			<joint name="${camera_name}_right_camera_optical_joint" type="fixed">
+				<origin xyz="0 0 0" rpy="-${M_PI/2} 0.0 -${M_PI/2}" />
+				<parent link="${camera_name}_${right_name}_${frame_suffix}" />
+				<child link="${camera_name}_${right_name}_${optical_frame_suffix}" />
+			</joint>
+		</xacro:if>
 	</xacro:macro>
 </robot>
