Commit message: Add script for converting depthai_boards descriptions to urdf and refactor urdf

File: depthai_descriptions/urdf/include/base_macro.urdf.xacro (robot description, xacro)
@@ -2,8 +2,10 @@
 <robot name="base"
 	xmlns:xacro="http://ros.org/wiki/xacro">
+	<xacro:include filename="$(find depthai_descriptions)/urdf/include/model_config.urdf.xacro" />
 	<xacro:macro name="base"
 		params="camera_name camera_model parent base_frame
                                            cam_pos_x cam_pos_y cam_pos_z
                                            cam_roll cam_pitch cam_yaw has_imu r:=0.8 g:=0.8 b:=0.8 a:=0.8 simulation:=false">
+		<xacro:depthai_model_config camera_model="${camera_model}" />
 		<xacro:if value="${simulation}">
 			<xacro:property
@@ -20,5 +22,4 @@
 		<!-- base_link of the sensor-->
 		<link name="${base_frame}" />
-		<xacro:property name="M_PI" value="3.1415926535897931" />
 		<xacro:property name="model" value="${camera_model}" />
 		<joint name="${camera_name}_center_joint" type="fixed">
@@ -29,30 +30,15 @@
 		</joint>
 		<!-- device Center -->
-		<xacro:unless value="${model in ['OAK-D-SR-POE']}">
-			<link name="${camera_name}_model_origin">
-				<visual>
-					<origin xyz="0 0 0" rpy="0 0 0" />
-					<geometry>
-						<mesh filename="${file_prefix}/urdf/models/${model}.stl" />
-					</geometry>
-					<material name="mat">
-						<color rgba="${r} ${g} ${b} ${a}" />
-					</material>
-				</visual>
-			</link>
-		</xacro:unless>
-		<xacro:if value="${model in ['OAK-D-SR-POE']}">
-			<link name="${camera_name}_model_origin">
-				<visual>
-					<origin xyz="0.019 0 0" rpy="0 0 0" />
-					<geometry>
-						<mesh filename="${file_prefix}/urdf/models/${model}.stl" />
-					</geometry>
-					<material name="mat">
-						<color rgba="${r} ${g} ${b} ${a}" />
-					</material>
-				</visual>
-			</link>
-		</xacro:if>
+		<link name="${camera_name}_model_origin">
+			<visual>
+				<origin xyz="${device_config['mesh_xyz']}" rpy="0 0 0" />
+				<geometry>
+					<mesh filename="${file_prefix}/urdf/models/${model}.stl" />
+				</geometry>
+				<material name="mat">
+					<color rgba="${r} ${g} ${b} ${a}" />
+				</material>
+			</visual>
+		</link>
 		<joint name="${camera_name}_model_origin_joint" type="fixed">
 			<parent link="${base_frame}" />
@@ -61,35 +47,15 @@
 		</joint>
 		<!-- IMU -->
-		<xacro:if value="${model == 'OAK-D'}">
-			<xacro:property name="imu_offset_x" value="0.0" />
-			<xacro:property name="imu_offset_y" value="-0.015" />
-			<xacro:property name="imu_offset_z" value="-0.013662" />
-			<xacro:property name="imu_r" value="0.0" />
-			<xacro:property name="imu_p" value="${M_PI/2.0}" />
-			<xacro:property name="imu_y" value="0.0" />
-		</xacro:if>
-		<xacro:if value="${model == 'OAK-D-PRO'}">
-			<xacro:property name="imu_offset_x" value="-0.008" />
-			<xacro:property name="imu_offset_y" value="-0.037945" />
-			<xacro:property name="imu_offset_z" value="-0.00079" />
-			<xacro:property name="imu_r" value="${M_PI}" />
-			<xacro:property name="imu_p" value="${M_PI/2.0}" />
-			<xacro:property name="imu_y" value="0.0" />
-		</xacro:if>
-		<xacro:if value="${model == 'OAK-D-POE'}">
-			<xacro:property name="imu_offset_x" value="-0.008" />
-			<xacro:property name="imu_offset_y" value="-0.04" />
-			<xacro:property name="imu_offset_z" value="-0.020265" />
-			<xacro:property name="imu_r" value="${M_PI}" />
-			<xacro:property name="imu_p" value="${M_PI/2.0}" />
-			<xacro:property name="imu_y" value="0.0" />
-		</xacro:if>
 		<xacro:if value="${has_imu}">
+			<xacro:if value="${device_config['imu_xyz'] is None or device_config['imu_rpy'] is None}">
+				<xacro:property name="invalid_imu" lazy_eval="false"
+					value="${xacro.fatal('No IMU transform defined for camera_model: ' + camera_model)}" />
+			</xacro:if>
 			<link name="${camera_name}_imu_frame" />
 			<joint name="${camera_name}_imu_joint" type="fixed">
 				<parent link="${base_frame}" />
 				<child link="${camera_name}_imu_frame" />
-				<origin xyz="${imu_offset_x} ${imu_offset_y} ${imu_offset_z}"
-					rpy="${imu_r} ${imu_p} ${imu_y}" />
+				<origin xyz="${device_config['imu_xyz']}"
+					rpy="${device_config['imu_rpy']}" />
 			</joint>
 		</xacro:if>

File: depthai_descriptions/urdf/include/depthai_macro.urdf.xacro (robot description, xacro)
@@ -2,4 +2,21 @@
 <robot name="depthai_camera"
 	xmlns:xacro="http://ros.org/wiki/xacro">
+	<!-- Camera and optical frames share the same structure for every sensor. -->
+	<xacro:macro name="depthai_camera_frame"
+		params="camera_name base_frame sensor_name joint_name xyz frame_suffix optical_frame_suffix">
+		<xacro:property name="M_PI" value="3.1415926535897931" />
+		<link name="${camera_name}_${sensor_name}_${frame_suffix}" />
+		<joint name="${camera_name}_${joint_name}_camera_joint" type="fixed">
+			<parent link="${base_frame}" />
+			<child link="${camera_name}_${sensor_name}_${frame_suffix}" />
+			<origin xyz="${xyz}" rpy="0 0 0" />
+		</joint>
+		<link name="${camera_name}_${sensor_name}_${optical_frame_suffix}" />
+		<joint name="${camera_name}_${joint_name}_camera_optical_joint" type="fixed">
+			<origin xyz="0 0 0" rpy="-${M_PI/2} 0.0 -${M_PI/2}" />
+			<parent link="${camera_name}_${sensor_name}_${frame_suffix}" />
+			<child link="${camera_name}_${sensor_name}_${optical_frame_suffix}" />
+		</joint>
+	</xacro:macro>
 	<xacro:macro name="depthai_camera"
 		params="camera_name camera_model parent base_frame
@@ -7,8 +24,5 @@
                                            cam_roll cam_pitch cam_yaw r:=0.8 g:=0.8 b:=0.8 a:=0.8 simulation:=false rs_compat:=false">
 		<xacro:include filename="$(find depthai_descriptions)/urdf/include/base_macro.urdf.xacro" />
-		<xacro:property name="M_PI" value="3.1415926535897931" />
-		<xacro:property name="model" value="${camera_model}" />
-		<xacro:property name="has_imu" value="false" />
-		<xacro:property name="baseline" value="0.075" />
+		<xacro:depthai_model_config camera_model="${camera_model}" />
 		<xacro:if value="${rs_compat}">
 			<xacro:property name="frame_suffix" value="frame" />
@@ -25,128 +39,22 @@
 			<xacro:property name="right_name" value="right" />
 		</xacro:unless>
-		<xacro:if value="${model in ['OAK-D-SR']}">
-			<xacro:property name="baseline" value="0.02" />
-		</xacro:if>
-		<xacro:if value="${model in ['OAK-D', 'OAK-D-PRO', 'OAK-D-POE']}">
-			<xacro:property name="has_imu" value="true" />
-		</xacro:if>
 		<xacro:base camera_name="${camera_name}" parent="${parent}" camera_model="${camera_model}"
 			base_frame="${base_frame}" cam_pos_x="${cam_pos_x}" cam_pos_y="${cam_pos_y}"
 			cam_pos_z="${cam_pos_z}" cam_roll="${cam_roll}" cam_pitch="${cam_pitch}"
-			cam_yaw="${cam_yaw}" has_imu="${has_imu}" simulation="${simulation}" />
-		<!-- RGB Camera -->
-		<xacro:unless value="${model in ['OAK-D-SR']}">
-			<link name="${camera_name}_${rgb_name}_${frame_suffix}" />
-			<joint name="${camera_name}_rgb_camera_joint" type="fixed">
-				<parent link="${base_frame}" />
-				<child link="${camera_name}_${rgb_name}_${frame_suffix}" />
-				<origin xyz="0 0 0" rpy="0 0 0" />
-			</joint>
-			<link name="${camera_name}_${rgb_name}_${optical_frame_suffix}" />
-			<joint name="${camera_name}_rgb_camera_optical_joint" type="fixed">
-				<origin xyz="0 0 0" rpy="-${M_PI/2} 0.0 -${M_PI/2}" />
-				<parent link="${camera_name}_${rgb_name}_${frame_suffix}" />
-				<child link="${camera_name}_${rgb_name}_${optical_frame_suffix}" />
-			</joint>
-		</xacro:unless>
-		<!-- LR and SR POE have different baselines and positions -->
-		<xacro:unless value="${model in ['OAK-D-LR', 'OAK-D-SR-POE', 'OAK-T']}">
-			<!-- Left Camera -->
-			<link name="${camera_name}_${left_name}_${frame_suffix}" />
-			<joint name="${camera_name}_left_camera_joint" type="fixed">
-				<parent link="${base_frame}" />
-				<child link="${camera_name}_${left_name}_${frame_suffix}" />
-				<origin xyz="0 ${baseline/2} 0" rpy="0 0 0" />
-			</joint>
-			<link name="${camera_name}_${left_name}_${optical_frame_suffix}" />
-			<joint name="${camera_name}_left_camera_optical_joint" type="fixed">
-				<origin xyz="0 0 0" rpy="-${M_PI/2} 0.0 -${M_PI/2}" />
-				<parent link="${camera_name}_${left_name}_${frame_suffix}" />
-				<child link="${camera_name}_${left_name}_${optical_frame_suffix}" />
-			</joint>
-			<!-- right Camera -->
-			<link name="${camera_name}_${right_name}_${frame_suffix}" />
-			<joint name="${camera_name}_right_camera_joint" type="fixed">
-				<parent link="${base_frame}" />
-				<child link="${camera_name}_${right_name}_${frame_suffix}" />
-				<origin xyz="0 -${baseline/2} 0" rpy="0 0 0" />
-			</joint>
-			<link name="${camera_name}_${right_name}_${optical_frame_suffix}" />
-			<joint name="${camera_name}_right_camera_optical_joint" type="fixed">
-				<origin xyz="0 0 0" rpy="-${M_PI/2} 0.0 -${M_PI/2}" />
-				<parent link="${camera_name}_${right_name}_${frame_suffix}" />
-				<child link="${camera_name}_${right_name}_${optical_frame_suffix}" />
-			</joint>
-		</xacro:unless>
-		<xacro:if value="${model in ['OAK-D-LR']}">
-			<!-- left Camera -->
-			<link name="${camera_name}_${left_name}_${frame_suffix}" />
-			<joint name="${camera_name}_left_camera_joint" type="fixed">
-				<parent link="${base_frame}" />
-				<child link="${camera_name}_${left_name}_${frame_suffix}" />
-				<origin xyz="0 0.1 0" rpy="0 0 0" />
-			</joint>
-			<link name="${camera_name}_${left_name}_${optical_frame_suffix}" />
-			<joint name="${camera_name}_left_camera_optical_joint" type="fixed">
-				<origin xyz="0 0 0" rpy="-${M_PI/2} 0.0 -${M_PI/2}" />
-				<parent link="${camera_name}_${left_name}_${frame_suffix}" />
-				<child link="${camera_name}_${left_name}_${optical_frame_suffix}" />
-			</joint>
-			<!-- right Camera -->
-			<link name="${camera_name}_${right_name}_${frame_suffix}" />
-			<joint name="${camera_name}_right_camera_joint" type="fixed">
-				<parent link="${base_frame}" />
-				<child link="${camera_name}_${right_name}_${frame_suffix}" />
-				<origin xyz="0 -0.05 0" rpy="0 0 0" />
-			</joint>
-			<link name="${camera_name}_${right_name}_${optical_frame_suffix}" />
-			<joint name="${camera_name}_right_camera_optical_joint" type="fixed">
-				<origin xyz="0 0 0" rpy="-${M_PI/2} 0.0 -${M_PI/2}" />
-				<parent link="${camera_name}_${right_name}_${frame_suffix}" />
-				<child link="${camera_name}_${right_name}_${optical_frame_suffix}" />
-			</joint>
+			cam_yaw="${cam_yaw}" has_imu="${device_config['imu_xyz'] is not None}" simulation="${simulation}" />
+		<xacro:if value="${device_config['rgb_xyz'] is not None}">
+			<xacro:depthai_camera_frame camera_name="${camera_name}" base_frame="${base_frame}"
+				sensor_name="${rgb_name}" joint_name="rgb" xyz="${device_config['rgb_xyz']}"
+				frame_suffix="${frame_suffix}" optical_frame_suffix="${optical_frame_suffix}" />
 		</xacro:if>
-		<xacro:if value="${model in ['OAK-D-SR-POE']}">
-			<!-- left Camera -->
-			<link name="${camera_name}_${left_name}_${frame_suffix}" />
-			<joint name="${camera_name}_left_camera_joint" type="fixed">
-				<parent link="${base_frame}" />
-				<child link="${camera_name}_${left_name}_${frame_suffix}" />
-				<origin xyz="0 0.0375 0" rpy="0 0 0" />
-			</joint>
-			<link name="${camera_name}_${left_name}_${optical_frame_suffix}" />
-			<joint name="${camera_name}_left_camera_optical_joint" type="fixed">
-				<origin xyz="0 0 0" rpy="-${M_PI/2} 0.0 -${M_PI/2}" />
-				<parent link="${camera_name}_${left_name}_${frame_suffix}" />
-				<child link="${camera_name}_${left_name}_${optical_frame_suffix}" />
-			</joint>
-			<!-- right Camera -->
-			<link name="${camera_name}_${right_name}_${frame_suffix}" />
-			<joint name="${camera_name}_right_camera_joint" type="fixed">
-				<parent link="${base_frame}" />
-				<child link="${camera_name}_${right_name}_${frame_suffix}" />
-				<origin xyz="0 0.0175 0" rpy="0 0 0" />
-			</joint>
-			<link name="${camera_name}_${right_name}_${optical_frame_suffix}" />
-			<joint name="${camera_name}_right_camera_optical_joint" type="fixed">
-				<origin xyz="0 0 0" rpy="-${M_PI/2} 0.0 -${M_PI/2}" />
-				<parent link="${camera_name}_${right_name}_${frame_suffix}" />
-				<child link="${camera_name}_${right_name}_${optical_frame_suffix}" />
-			</joint>
+		<xacro:if value="${device_config['left_xyz'] is not None}">
+			<xacro:depthai_camera_frame camera_name="${camera_name}" base_frame="${base_frame}"
+				sensor_name="${left_name}" joint_name="left" xyz="${device_config['left_xyz']}"
+				frame_suffix="${frame_suffix}" optical_frame_suffix="${optical_frame_suffix}" />
 		</xacro:if>
-		<xacro:if value="${model in ['OAK-T']}">
-			<!-- right Camera -->
-			<link name="${camera_name}_cam_e_${frame_suffix}" />
-			<joint name="${camera_name}_right_camera_joint" type="fixed">
-				<parent link="${base_frame}" />
-				<child link="${camera_name}_cam_e_${frame_suffix}" />
-				<origin xyz="0 -0.025 0" rpy="0 0 0" />
-			</joint>
-			<link name="${camera_name}_cam_e_${optical_frame_suffix}" />
-			<joint name="${camera_name}_right_camera_optical_joint" type="fixed">
-				<origin xyz="0 0 0" rpy="-${M_PI/2} 0.0 -${M_PI/2}" />
-				<parent link="${camera_name}_cam_e_${frame_suffix}" />
-				<child link="${camera_name}_cam_e_${optical_frame_suffix}" />
-			</joint>
+		<xacro:if value="${device_config['right_xyz'] is not None}">
+			<xacro:depthai_camera_frame camera_name="${camera_name}" base_frame="${base_frame}"
+				sensor_name="${device_config['right_name'] or right_name}" joint_name="right" xyz="${device_config['right_xyz']}"
+				frame_suffix="${frame_suffix}" optical_frame_suffix="${optical_frame_suffix}" />
 		</xacro:if>
 	</xacro:macro>

Commit message: Simplify diff

File: depthai_descriptions/urdf/include/base_macro.urdf.xacro (robot description, xacro)
@@ -27,5 +27,4 @@
 		<!-- base_link of the sensor-->
 		<link name="${base_frame}" />
-		<xacro:property name="model" value="${camera_model}" />
 		<joint name="${camera_name}_center_joint" type="fixed">
 			<parent link="${parent}" />
